File: IGBT DRIVER.kicad_pcb (KiCad board)
At the start: 2 copper layers, 139.2 x 61 mm, 150 parts, among them J6 Conn_01x02, J7 Conn_01x02, Q1 BC817, Q10 BC817, Q11 BC817, Q12 BC817, Q13 BC817, Q14 BC807, Q15 BC817, Q16 BC817, Q17 BC807, Q18 BC817, Q19 TIP41, Q2 BC817, Q20 TIP42, Q3 BC817, Q4 BC807, Q5 BC817, Q6 BC817, Q7 BC817, Q8 TIP41, Q9 TIP42, U2 6N136S, U3 PC817, U4 6N136S, U5 PC817

Commit message: some placement
Parts:
- added C25: 1uF, Capacitor_SMD:C_1206_3216Metric_Pad1.33x1.80mm_HandSolder, F.Cu at (143.6, 29.0)
- added C26: 1uF, Capacitor_SMD:C_1206_3216Metric_Pad1.33x1.80mm_HandSolder, F.Cu at (151.7, 27.0)
- added C27: 1uF, Capacitor_SMD:C_1206_3216Metric_Pad1.33x1.80mm_HandSolder, F.Cu at (144.7, 32.3)
- added C28: 1uF, Capacitor_SMD:C_1206_3216Metric_Pad1.33x1.80mm_HandSolder, F.Cu at (150.7, 33.7)
- added C29: 1uF, Capacitor_SMD:C_1206_3216Metric_Pad1.33x1.80mm_HandSolder, F.Cu at (132.4, 47.1)
- added C30: 1uF, Capacitor_SMD:C_1206_3216Metric_Pad1.33x1.80mm_HandSolder, F.Cu at (167.9, 11.9)
- added C31: 1uF, Capacitor_SMD:C_1206_3216Metric_Pad1.33x1.80mm_HandSolder, F.Cu at (157.7, 21.4)
- added C32: 1uF, Capacitor_SMD:C_1206_3216Metric_Pad1.33x1.80mm_HandSolder, F.Cu at (165.4, 15.3)
- added C33: 1uF, Capacitor_SMD:C_1206_3216Metric_Pad1.33x1.80mm_HandSolder, F.Cu at (151.7, 23.6)
- added C34: 1uF, Capacitor_SMD:C_1206_3216Metric_Pad1.33x1.80mm_HandSolder, F.Cu at (144.5, 39.0)
- added C35: 1uF, Capacitor_SMD:C_1206_3216Metric_Pad1.33x1.80mm_HandSolder, F.Cu at (138.4, 44.8)
- added C36: 1uF, Capacitor_SMD:C_1206_3216Metric_Pad1.33x1.80mm_HandSolder, F.Cu at (157.7, 28.1)
- added C37: 1uF, Capacitor_SMD:C_1206_3216Metric_Pad1.33x1.80mm_HandSolder, F.Cu at (163.7, 22.0)
- added C38: 1uF, Capacitor_SMD:C_1206_3216Metric_Pad1.33x1.80mm_HandSolder, F.Cu at (138.4, 48.2)
- added C39: 1uF, Capacitor_SMD:C_1206_3216Metric_Pad1.33x1.80mm_HandSolder, F.Cu at (175.9, 7.57)
- added C40: 1uF, Capacitor_SMD:C_1206_3216Metric_Pad1.33x1.80mm_HandSolder, F.Cu at (156.8, 31.5)
- added C41: 1uF, Capacitor_SMD:C_1206_3216Metric_Pad1.33x1.80mm_HandSolder, F.Cu at (188.2, 184.0)
- added C42: 1uF, Capacitor_SMD:C_1206_3216Metric_Pad1.33x1.80mm_HandSolder, F.Cu at (183.1, 184.0)
- added C43: 1uF, Capacitor_SMD:C_1206_3216Metric_Pad1.33x1.80mm_HandSolder, F.Cu at (188.2, 181.5)
- added C44: 1uF, Capacitor_SMD:C_1206_3216Metric_Pad1.33x1.80mm_HandSolder, F.Cu at (183.1, 181.5)
- added C45: 1uF, Capacitor_SMD:C_1206_3216Metric_Pad1.33x1.80mm_HandSolder, F.Cu at (188.2, 178.9)
- added C46: 1uF, Capacitor_SMD:C_1206_3216Metric_Pad1.33x1.80mm_HandSolder, F.Cu at (183.1, 178.9)
- added C47: 1uF, Capacitor_SMD:C_1206_3216Metric_Pad1.33x1.80mm_HandSolder, F.Cu at (188.2, 176.4)
- added C48: 1uF, Capacitor_SMD:C_1206_3216Metric_Pad1.33x1.80mm_HandSolder, F.Cu at (183.1, 176.4)
- added C49: 1uF, Capacitor_SMD:C_1206_3216Metric_Pad1.33x1.80mm_HandSolder, F.Cu at (188.2, 173.9)
- added C50: 1uF, Capacitor_SMD:C_1206_3216Metric_Pad1.33x1.80mm_HandSolder, F.Cu at (183.1, 173.9)
- added C51: 1uF, Capacitor_SMD:C_1206_3216Metric_Pad1.33x1.80mm_HandSolder, F.Cu at (188.2, 171.1)
- added C52: 1uF, Capacitor_SMD:C_1206_3216Metric_Pad1.33x1.80mm_HandSolder, F.Cu at (183.1, 171.1)
- added C53: 1uF, Capacitor_SMD:C_1206_3216Metric_Pad1.33x1.80mm_HandSolder, F.Cu at (188.2, 168.5)
- added C54: 1uF, Capacitor_SMD:C_1206_3216Metric_Pad1.33x1.80mm_HandSolder, F.Cu at (183.1, 168.5)
- added C55: 1uF, Capacitor_SMD:C_1206_3216Metric_Pad1.33x1.80mm_HandSolder, F.Cu at (188.2, 166.0)
- added C56: 1uF, Capacitor_SMD:C_1206_3216Metric_Pad1.33x1.80mm_HandSolder, F.Cu at (183.1, 166.0)
- added C57: 1uF, Capacitor_SMD:C_1206_3216Metric_Pad1.33x1.80mm_HandSolder, F.Cu at (188.2, 163.5)
- added C58: 1uF, Capacitor_SMD:C_1206_3216Metric_Pad1.33x1.80mm_HandSolder, F.Cu at (183.1, 163.5)
- added F1: Fuse_Small, IGBT-DRIVER-emad:fuse.holder.1808, F.Cu at (189.5, 12.7)
- added F2: Fuse, Fuse:Fuse_Schurter_UMZ250, F.Cu at (104.0, 42.7)
- added F3: Fuse_Small, IGBT-DRIVER-emad:fuse.holder.1808, F.Cu at (110.0, 18.7)
- added F4: Fuse, Fuse:Fuse_Schurter_UMZ250, F.Cu at (163.2, 267.4)
- added F6: Fuse_Small, IGBT-DRIVER-emad:fuse.holder.1808, F.Cu at (222.5, 183.8)
- added H5: MountingHole, MountingHole:MountingHole_4.3x6.2mm_M4_Pad_Via, F.Cu at (203.6, 24.3)
- added J1: Conn_02x05_Odd_Even, Connector_IDC:IDC-Header_2x05-1MP_P2.54mm_Latch_Horizontal, F.Cu at (102.0, 165.4)
- added J3: Screw_Terminal_01x01, IGBT-DRIVER-emad:COOLERI, F.Cu at (199.1, 10.3)
- added J5: Screw_Terminal_01x01, IGBT-DRIVER-emad:COOLERI, F.Cu at (198.3, 18.5)
- added L2: 10uh, Inductor_SMD:L_12x12mm_H6mm, F.Cu at (191.0, 4.78)
- added R1: 1.8k, Resistor_SMD:R_0805_2012Metric, F.Cu at (218.9, 9.08)
- added R11: 1K, Resistor_SMD:R_0805_2012Metric, F.Cu at (173.4, 21.8)
- added R12: 1k, Resistor_SMD:R_0805_2012Metric, F.Cu at (112.4, 314.1)
- added R13: 3.3K, Resistor_SMD:R_0805_2012Metric, F.Cu at (95.9, 314.2)
- added R18: 1K, Resistor_SMD:R_0805_2012Metric, F.Cu at (108.0, 312.9)
- added R19: 1K, Resistor_SMD:R_0805_2012Metric, F.Cu at (131.7, 290.3)
- added R2: 1k, Resistor_SMD:R_0805_2012Metric, F.Cu at (139.7, 13.4)
- added R21: 10K, Resistor_SMD:R_0805_2012Metric, F.Cu at (214.1, 170.6)
- added R22: 1K, Resistor_SMD:R_0805_2012Metric, F.Cu at (131.7, 293.3)
- added R3: 1.8k, Resistor_SMD:R_0805_2012Metric, F.Cu at (238.8, 12.4)
- added R5: 3.3K, Resistor_SMD:R_0805_2012Metric, F.Cu at (131.6, 50.3)
- added R8: 1K, Resistor_SMD:R_0805_2012Metric, F.Cu at (143.7, 48.9)
- added R9: 1K, Resistor_SMD:R_0805_2012Metric, F.Cu at (167.3, 26.3)
- added RClamp1: 10K, Resistor_SMD:R_0805_2012Metric, F.Cu at (167.3, 29.3)
- added Roff3: 40, Resistor_SMD:R_2512_6332Metric, F.Cu at (122.5, 24.4)
- added Roff4: 40, Resistor_SMD:R_2512_6332Metric, F.Cu at (206.1, 175.8)
- added Ron3: 40, Resistor_SMD:R_2512_6332Metric, F.Cu at (206.1, 167.9)
- added Ron4: 40, Resistor_SMD:R_2512_6332Metric, F.Cu at (158.1, 13.0)
- added U1: miw06-24s24, IGBT-DRIVER-emad:MIWI06, F.Cu at (153.8, 180.6)
- added U6: miw06-24s24, IGBT-DRIVER-emad:MIWI06, F.Cu at (153.6, 140.3)
- C1, C22, C24, C6, CShortPulseFilter1, CblankTime1, Cex1, Cex2, Cex3, Cex4, Cex5, Cex6, Cex7, CsoftTurnOff2, CsoftTurnOffTiming1: footprint Capacitor_SMD:C_1206_3216Metric_Pad1.33x1.80mm_HandSolder -> Capacitor_SMD:C_0805_2012Metric
- C10, C2: value 47uf/35v -> 1uF; footprint Capacitor_THT:CP_Radial_D8.0mm_P3.80mm -> Capacitor_SMD:C_1206_3216Metric_Pad1.33x1.80mm_HandSolder
- C12, CDynamic1: footprint Capacitor_THT:C_Disc_D16.0mm_W5.0mm_P10.00mm -> Capacitor_THT:C_Rect_L16.5mm_W6.0mm_P15.00mm_MKT
- C14: footprint Capacitor_SMD:C_1206_3216Metric_Pad1.33x1.80mm_HandSolder -> Capacitor_SMD:C_0805_2012Metric; moved to B.Cu
- Cclamp1, Cclamp2: footprint Capacitor_SMD:C_1206_3216Metric -> Capacitor_SMD:C_0805_2012Metric
- D11, D4: value 1.5KE13A -> 1.5KE14A; footprint Diode_THT:D_DO-201AD_P5.08mm_Vertical_AnodeUp -> Diode_THT:D_DO-201AD_P15.24mm_Horizontal
- D12, D13, D16, D17, D18, D19, D20, D21, D5, D6, DStatic1, DStatic2, DStatic3, DStatic4, DStatic5, DzDynamic1: footprint Diode_THT:D_DO-201AD_P5.08mm_Vertical_AnodeUp -> Diode_THT:D_DO-201AD_P15.24mm_Horizontal
- H1, H2, H3, H4: footprint TestPoint:TestPoint_Plated_Hole_D4.0mm -> MountingHole:MountingHole_4.3x6.2mm_M4_Pad_Via
- Q14, Q16: moved to B.Cu
- Q19, Q8: value TIP41 -> d44vh10; footprint Package_TO_SOT_THT:TO-220-3_Vertical -> Package_TO_SOT_SMD:TO-252-2
- Q20, Q9: value TIP42 -> D45VH10; footprint Package_TO_SOT_THT:TO-220-3_Vertical -> Package_TO_SOT_SMD:TO-252-2
- R15: footprint Resistor_THT:R_Axial_DIN0207_L6.3mm_D2.5mm_P10.16mm_Horizontal -> Resistor_SMD:R_0805_2012Metric; moved to B.Cu
- RAfterfaultTurnOnDelay1, RBlankTime1, RSofTurnoffTiming1, Rex1, Rex10, Rex11, Rex12, Rex13, Rex15, Rex16, Rex17, Rex18, Rex2, Rex3, Rex4, Rex6, Rex7, Rex8, Rex9, RshortPulseFilter1, RsoftTurnoff2: footprint Resistor_THT:R_Axial_DIN0207_L6.3mm_D2.5mm_P10.16mm_Horizontal -> Resistor_SMD:R_0805_2012Metric
- Roff1, Roff2, Ron1, Ron2: value 20 -> 40; footprint Resistor_THT:R_Axial_DIN0207_L6.3mm_D2.5mm_P10.16mm_Horizontal -> Resistor_SMD:R_2512_6332Metric
- moved Rex15 369.7 mm to (50.0, 313.6)
- moved D11 369.6 mm to (50.8, 271.8)
- moved Rex9 354.7 mm to (50.0, 305.5)
- moved Rex12 349.9 mm to (50.0, 309.6)
- moved C6 347.3 mm to (102.7, 308.8)
- moved Cex7 343.2 mm to (108.8, 303.0)
- moved H4 341.0 mm to (101.2, 184.1)
- moved Q11 340.0 mm to (114.1, 305.0)
- moved Q17 338.7 mm to (113.6, 310.3)
- moved Dex6 336.7 mm to (109.0, 289.0)
- moved Rex11 329.0 mm to (50.0, 297.4)
- moved U4 327.8 mm to (81.7, 301.2)
- moved C23 320.5 mm to (91.3, 300.1)
- moved Rex10 318.9 mm to (84.0, 283.9)
- moved Dex10 318.2 mm to (89.7, 311.7)
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Connections:
- C10 pad 1: /EMITTER_BOTTOM -> /GND_top
- C10 pad 2: /GND_BOTTOM -> /EMITTER_TOP
- C16 pad 1: Net-(C16-Pad1) -> +15V
- C17 pad 2: Net-(C16-Pad1) -> +15V
- C2 pad 1: /EMITTER_TOP -> /GND_top
- C2 pad 2: /GND_top -> /VCC_top
- C4 pad 1: Net-(C4-Pad1) -> +15V
- C9 pad 2: Net-(C4-Pad1) -> +15V
- D1 pad 2: (no net) -> Net-(D1-Pad2)
- D12 pad 1: (no net) -> /GATE_BOTTOM
- D2 pad 1: (no net) -> /Pulse-TOP
- D2 pad 2: (no net) -> Net-(D2-Pad2)
- D22 pad 1: (no net) -> Net-(D22-Pad1)
- D29 pad 2: (no net) -> Net-(D29-Pad2)
- D29 pad 4: +15V -> Net-(D29-Pad4)
- D6 pad 1: (no net) -> /GATE_TOP
- D8 pad 1: (no net) -> /Pulse-BOTTOM
- D8 pad 2: (no net) -> Net-(D8-Pad2)
- D9 pad 2: (no net) -> Net-(D9-Pad2)
- DZunderVoltageFault1 pad 1: (no net) -> Net-(DZunderVoltageFault1-Pad1)
- Q15 pad 1: (no net) -> Net-(Q15-Pad1)
- Q17 pad 3: (no net) -> Net-(Q17-Pad3)
- Q6 pad 1: (no net) -> Net-(Q6-Pad1)
- QfaultLatch1 pad 3: (no net) -> Net-(QfaultLatch1-Pad3)
- U2 pad 2: (no net) -> Net-(R2-Pad1)
- U4 pad 2: (no net) -> Net-(R12-Pad1)
Routing:
- net /GATE_BOTTOM: track 0.00 -> 43.1 mm
- net Net-(Dex3-Pad2): track 0.00 -> 20.3 mm
- net /EMITTER_BOTTOM: track 0.00 -> 5.13 mm
Other:
- board size 139.2 x 61 mm -> 139.2 x 83.2 mm

Commit message: vg
Parts:
- added R20: 1k, Resistor_SMD:R_0805_2012Metric, F.Cu at (145.7, 316.4)
- added R23: 1k, Resistor_SMD:R_0805_2012Metric, F.Cu at (165.2, 316.4)
- U1, U6: value miw06-24s24 -> PC817; footprint IGBT-DRIVER-emad:MIWI06 -> Package_DIP:DIP-4_W7.62mm
- moved U6 176.7 mm to (153.7, 317.0)
- moved U1 137.8 mm to (134.3, 317.0)
- moved D11 137.5 mm to (160.1, 188.3)
- moved D13 124.9 mm to (154.4, 195.3), turned to 270 degrees
- moved Rex13 86.3 mm to (154.5, 189.6), turned to 90 degrees
- moved D16 76.3 mm to (162.6, 210.6), turned to 90 degrees
- moved D17 66.2 mm to (171.4, 210.3), turned to 90 degrees
- moved D18 55.6 mm to (179.7, 210.4), turned to 90 degrees
- moved D14 55.3 mm to (154.0, 241.5), turned to 180 degrees
- moved D19 46.0 mm to (188.8, 210.3), turned to 90 degrees
- moved D20 36.6 mm to (197.9, 210.3), turned to 90 degrees
- moved C12 29.3 mm to (204.8, 209.6), turned to 90 degrees
- moved R14 25.2 mm to (210.0, 207.5), turned to 90 degrees
- moved D21 0.19 mm to (215.4, 210.2)
Connections:
- Cex2 pad 2: /Reset_top -> /Gate Driver Top/Protection
- Cex6 pad 2: /Reset_BOTTOM -> /Gate Driver bottom/Protection
- D14 pad 2: /Reset_BOTTOM -> /Gate Driver bottom/Protection
- Dex2 pad 1: /Reset_top -> /Gate Driver Top/Protection
- Dex7 pad 1: /Reset_BOTTOM -> /Gate Driver bottom/Protection
- DzSaturation1 pad 2: /Reset_top -> /Gate Driver Top/Protection
- Q11 pad 1: /Reset_BOTTOM -> /Gate Driver bottom/Protection
- QsoftTurnOnn1 pad 1: /Reset_top -> /Gate Driver Top/Protection
- R13 pad 2: /Reset_BOTTOM -> /Gate Driver bottom/Protection
- R5 pad 2: /Reset_top -> /Gate Driver Top/Protection
- Rex14 pad 2: /Reset_BOTTOM -> /Gate Driver bottom/Protection
- Rex5 pad 2: /Reset_top -> /Gate Driver Top/Protection
- U1 pad 2: GNDD -> /Reset_top
- U1 pad 3: GNDD -> /Gate Driver Top/Protection
- U6 pad 2: GNDD -> /Reset_BOTTOM
- U6 pad 3: GNDD -> /Gate Driver bottom/Protection
Routing:
- net Net-(C12-Pad1): track 0.00 -> 30.0 mm
- net Net-(C12-Pad2): track 0.00 -> 28.7 mm
- net Net-(D19-Pad2): track 0.00 -> 21.0 mm
- net Net-(Dex3-Pad2): track 20.3 -> 0.00 mm
- net Net-(D12-Pad2): track 0.00 -> 14.1 mm
Other:
- outline, holes or cut-outs redrawn

Commit message: some placements have done
Parts:
- removed C1, C22, C24: 100nF, Capacitor_SMD:C_0805_2012Metric
- removed C10, C2, C25, C26, C27, C28, C29, C30, C31, C32, C33, C34, C35, C36, C37, C38, C39, C40: 1uF, Capacitor_SMD:C_1206_3216Metric_Pad1.33x1.80mm_HandSolder
- removed C21, C23: 47uf/35v, Capacitor_THT:CP_Radial_D8.0mm_P3.80mm
- removed C5: 1nF, Capacitor_SMD:C_1206_3216Metric_Pad1.33x1.80mm_HandSolder
- removed CDynamic1: 100nF, Capacitor_THT:C_Rect_L16.5mm_W6.0mm_P15.00mm_MKT
- removed CShortPulseFilter1, CblankTime1: 100pF, Capacitor_SMD:C_0805_2012Metric
- removed Cclamp1: C, Capacitor_SMD:C_0805_2012Metric
- removed Cex1: 96pF, Capacitor_SMD:C_0805_2012Metric
- removed Cex2: 1nF, Capacitor_SMD:C_0805_2012Metric
- removed CsoftTurnOff2: 10nF, Capacitor_SMD:C_0805_2012Metric
- removed CsoftTurnOffTiming1: 22nF, Capacitor_SMD:C_0805_2012Metric
- removed D11, D4: 1.5KE14A, Diode_THT:D_DO-201AD_P15.24mm_Horizontal
- removed D12, D6: 1.5KE6V8A, Diode_THT:D_DO-201AD_P15.24mm_Horizontal
- removed D16, D17, D18, D19, D20, D21, DStatic1, DStatic2, DStatic3, DStatic4, DStatic5, DzDynamic1: 1.5KE160A, Diode_THT:D_DO-201AD_P15.24mm_Horizontal
- removed D2: 1.5KE4A, Diode_THT:D_DO-201AD_P5.08mm_Vertical_AnodeUp
- removed D3: Dz8v, Diode_THT:D_DO-201AD_P5.08mm_Vertical_AnodeUp
- removed D5: BYV26E, Diode_THT:D_DO-201AD_P15.24mm_Horizontal
- removed D7: 26v TVS, Diode_SMD:D_MELF
- removed DZunderVoltageFault1: BZX85C20, Diode_SMD:D_MELF
- removed Dex1, Dex2, Dex5, DprotectionHigh1, DprotectionLow1: 1n4148, Diode_SMD:D_SMA
- removed DzSaturation1: Dz10v, Diode_THT:D_DO-201AD_P5.08mm_Vertical_AnodeUp
- removed F2: Fuse, Fuse:Fuse_Schurter_UMZ250
- removed F3: Fuse_Small, IGBT-DRIVER-emad:fuse.holder.1808
- removed H5: MountingHole, MountingHole:MountingHole_4.3x6.2mm_M4_Pad_Via
- removed Q1, Q2, Q3, Q5, Q6, Q7, QsoftTurnOnn1: BC817, Package_TO_SOT_SMD:SOT-23
- removed Q4, QfaultLatch1: BC807, Package_TO_SOT_SMD:SOT-23
- removed Q8: d44vh10, Package_TO_SOT_SMD:TO-252-2
- removed Q9: D45VH10, Package_TO_SOT_SMD:TO-252-2
- removed Qclamp1: BUK7880-55A, Package_TO_SOT_SMD:SOT-223-3_TabPin2
- removed R11, R8, R9: 1K, Resistor_SMD:R_0805_2012Metric
- removed R20, RSofTurnoffTiming1, Rex7: 1k, Resistor_SMD:R_0805_2012Metric
- removed R7: 220, Resistor_THT:R_Axial_DIN0207_L6.3mm_D2.5mm_P10.16mm_Horizontal
- removed RAfterfaultTurnOnDelay1, RBlankTime1, Rex3, Rex6: 2.2k, Resistor_SMD:R_0805_2012Metric
- removed RClamp1: 10K, Resistor_SMD:R_0805_2012Metric
- removed RDynamic1: 20K, Resistor_THT:R_Axial_DIN0207_L6.3mm_D2.5mm_P10.16mm_Horizontal
- removed Rex2: 56k, Resistor_SMD:R_0805_2012Metric
- removed Rex4: 220, Resistor_SMD:R_0805_2012Metric
- removed Rex5: 1k, Resistor_THT:R_Axial_DIN0207_L6.3mm_D2.5mm_P10.16mm_Horizontal
- removed Roff1, Roff3, Ron1, Ron4: 40, Resistor_SMD:R_2512_6332Metric
- removed RshortPulseFilter1: 120, Resistor_SMD:R_0805_2012Metric
- removed RsoftTurnoff2: 10, Resistor_SMD:R_0805_2012Metric
- removed U2: 6N136S, Package_DIP:SMDIP-8_W9.53mm
- removed U3: PC817, Package_DIP:DIP-4_W7.62mm
- added D23: SMCJ160CA-13-F, IGBT-DRIVER-emad:DIOM7959X250N, B.Cu at (201.4, 200.4)
- added D24: SMCJ160CA-13-F, IGBT-DRIVER-emad:DIOM7959X250N, F.Cu at (201.4, 200.4)
- added D25: SMCJ160CA-13-F, IGBT-DRIVER-emad:DIOM7959X250N, F.Cu at (208.8, 200.3)
- added D26: SMCJ160CA-13-F, IGBT-DRIVER-emad:DIOM7959X250N, B.Cu at (208.8, 200.3)
- added D27: SMCJ160CA-13-F, IGBT-DRIVER-emad:DIOM7959X250N, B.Cu at (216.3, 200.3)
- added D28: SMCJ160CA-13-F, IGBT-DRIVER-emad:DIOM7959X250N, F.Cu at (216.3, 200.3)
- added U7: miw06-24s24, IGBT-DRIVER-emad:MIWI06, F.Cu at (154.1, 174.6)
- added U8: miw06-24s24, IGBT-DRIVER-emad:MIWI06, F.Cu at (153.9, 148.6)
- C12: value 100nF -> 100nF 250v; footprint Capacitor_THT:C_Rect_L16.5mm_W6.0mm_P15.00mm_MKT -> Capacitor_THT:C_Rect_L13.0mm_W4.0mm_P10.00mm_FKS3_FKP3_MKS4
- C15, C6, Cex3, Cex7, D22, Dex6, Dex7, Q12, Q13, Q15, Q17, Q18, Qclamp2, R13, R18, R19, R22, Rex10, Rex15, Rex16, Rex17, Rex18, Rex8: moved to B.Cu
- D10: footprint Diode_THT:D_DO-201AD_P5.08mm_Vertical_AnodeUp -> Diode_SMD:D_MELF; moved to B.Cu
- D13: footprint Diode_THT:D_DO-201AD_P15.24mm_Horizontal -> Diode_THT:D_DO-35_SOD27_P7.62mm_Horizontal
- D14: footprint Diode_THT:D_DO-201AD_P5.08mm_Vertical_AnodeUp -> Diode_SMD:D_MELF
- D15: value 26v TVS -> 26v Zener; moved to B.Cu
- F4: footprint Fuse:Fuse_Schurter_UMZ250 -> IGBT-DRIVER-emad:fuse.holder.1808
- R16: value 3.3k-1/4W -> 1.8k; footprint Resistor_THT:R_Axial_DIN0207_L6.3mm_D2.5mm_P10.16mm_Horizontal -> Resistor_SMD:R_0805_2012Metric; moved to B.Cu
- R2: value 1k -> 6k; footprint Resistor_SMD:R_0805_2012Metric -> Resistor_SMD:R_1206_3216Metric; moved to B.Cu
- R4: value 2k/1w -> 6k; footprint Resistor_THT:R_Axial_DIN0414_L11.9mm_D4.5mm_P7.62mm_Vertical -> Resistor_SMD:R_1206_3216Metric; moved to B.Cu
- R5: value 3.3K -> 6k; footprint Resistor_SMD:R_0805_2012Metric -> Resistor_SMD:R_1206_3216Metric; moved to B.Cu
- R6: value 3.3k-1/4W -> 1.5k; footprint Resistor_THT:R_Axial_DIN0207_L6.3mm_D2.5mm_P10.16mm_Horizontal -> Resistor_SMD:R_0805_2012Metric; moved to B.Cu
- Rex1: value 6.8k -> 1k; moved to B.Cu
- Rex14: footprint Resistor_THT:R_Axial_DIN0207_L6.3mm_D2.5mm_P10.16mm_Horizontal -> Resistor_SMD:R_0805_2012Metric
- U1: value PC817 -> ps2801; footprint Package_DIP:DIP-4_W7.62mm -> Package_SO:SOP-4_4.4x2.6mm_P1.27mm; moved to B.Cu
- U5, U6: value PC817 -> ps2801; footprint Package_DIP:DIP-4_W7.62mm -> Package_SO:SOP-4_4.4x2.6mm_P1.27mm
- moved H1 210.8 mm to (179.3, 207.5)
- moved R10 205.7 mm to (140.2, 197.1), turned to 180 degrees
- moved Dex10 195.3 mm to (220.7, 166.9), turned to 90 degrees
- moved F1 194.4 mm to (101.3, 185.9)
- moved D29 190.1 mm to (116.1, 163.6)
- moved C9 187.3 mm to (109.5, 141.8)
- moved J5 186.8 mm to (197.1, 205.2), turned to 90 degrees
- moved C16 181.1 mm to (134.1, 170.0), turned to 270 degrees
- moved R3 177.2 mm to (123.9, 147.3)
- moved U5 177.0 mm to (173.0, 160.8), turned to 270 degrees
- moved R1 175.4 mm to (116.1, 151.2)
- moved C19 175.3 mm to (123.4, 140.5)
- moved R6 172.2 mm to (186.2, 173.5), turned to 180 degrees
- moved C13 169.8 mm to (174.2, 174.4), turned to 180 degrees
- moved Rex15 168.6 mm to (173.9, 199.2), turned to 270 degrees
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Connections:
- C41 pad 2: /VCC_BOTTOM -> /Gate Driver bottom/Vpp
- C43 pad 2: /VCC_BOTTOM -> /Gate Driver bottom/Vpp
- C45 pad 2: /VCC_BOTTOM -> /Gate Driver bottom/Vpp
- C47 pad 2: /VCC_BOTTOM -> /Gate Driver bottom/Vpp
- C49 pad 2: /VCC_BOTTOM -> /Gate Driver bottom/Vpp
- C51 pad 2: /VCC_BOTTOM -> /Gate Driver bottom/Vpp
- C53 pad 2: /VCC_BOTTOM -> /Gate Driver bottom/Vpp
- C55 pad 2: /VCC_BOTTOM -> /Gate Driver bottom/Vpp
- C57 pad 2: /VCC_BOTTOM -> /Gate Driver bottom/Vpp
- D15 pad 1: /VCC_BOTTOM -> /Gate Driver bottom/Vpp
- Dex3 pad 1: /VCC_BOTTOM -> /Gate Driver bottom/Vpp
- F4 pad 1: /VCC_BOTTOM -> /Gate Driver bottom/Vpp
- F4 pad 2: (no net) -> /VCC_BOTTOM
- J1 pad 2: /Reset_top -> (no net)
- J1 pad 4: /Pulse-TOP -> (no net)
- J1 pad 8: /Error_top -> (no net)
- J3 pad 1: /Gate Driver Top/Collector -> Net-(J3-Pad1)
- J6 pad 1: /GATE_TOP -> (no net)
- J6 pad 2: /EMITTER_TOP -> (no net)
- Q11 pad 3: /Error_BOTTOM -> /Gate Driver bottom/fault
- Q16 pad 3: /VCC_BOTTOM -> /Gate Driver bottom/Vpp
- Q17 pad 1: /Error_BOTTOM -> /Gate Driver bottom/fault
- Q17 pad 2: /VCC_BOTTOM -> /Gate Driver bottom/Vpp
- Q19 pad 2: /VCC_BOTTOM -> /Gate Driver bottom/Vpp
- R16 pad 1: /VCC_BOTTOM -> Net-(R16-Pad1)
- R17 pad 2: Net-(D12-Pad2) -> /GATE_BOTTOM
- R19 pad 1: /VCC_BOTTOM -> /Gate Driver bottom/Vpp
- R2 pad 1: Net-(R2-Pad1) -> /GND_BOTTOM
- R2 pad 2: Net-(D2-Pad2) -> /VCC_BOTTOM
- R5 pad 1: Net-(QfaultLatch1-Pad3) -> /GND_BOTTOM
- R5 pad 2: /Gate Driver Top/Protection -> /VCC_BOTTOM
- R6 pad 1: /VCC_top -> /Gate Driver bottom/Vpp
- R6 pad 2: Net-(Dex2-Pad2) -> Net-(R16-Pad1)
- Rex1 pad 1: /EMITTER_TOP -> Net-(Rex1-Pad1)
- Rex1 pad 2: /VCC_top -> /Gate Driver bottom/fault
- Rex10 pad 2: /VCC_BOTTOM -> /Gate Driver bottom/Vpp
- Rex11 pad 2: /VCC_BOTTOM -> /Gate Driver bottom/Vpp
- Rex15 pad 1: /Error_BOTTOM -> /Gate Driver bottom/fault
- Rex16 pad 1: /VCC_BOTTOM -> /Gate Driver bottom/Vpp
- Rex17 pad 1: /VCC_BOTTOM -> /Gate Driver bottom/Vpp
- Rex18 pad 2: /VCC_BOTTOM -> /Gate Driver bottom/Vpp
- Rex8 pad 2: /VCC_BOTTOM -> /Gate Driver bottom/Vpp
- U1 pad 1: Net-(R20-Pad1) -> Net-(Rex1-Pad1)
- U1 pad 2: /Reset_top -> /GND_BOTTOM
- U1 pad 3: /Gate Driver Top/Protection -> /Vin-
- U1 pad 4: /GND_top -> /Error_BOTTOM
- U5 pad 1: /On_TOP -> (no net)
Routing:
- net Net-(C12-Pad1): track 30.0 -> 0.00 mm, vias 0 -> 10
- net Net-(C12-Pad2): track 28.7 -> 0.26 mm
- net /EMITTER_BOTTOM: track 5.13 -> 28.9 mm
- net Net-(D19-Pad2): track 21.0 -> 0.00 mm
- net Net-(D26-PadA): track 0.00 -> 14.8 mm
- net /GND_BOTTOM: track 0.00 -> 14.4 mm
- net Net-(D12-Pad2): track 14.1 -> 0.00 mm
- net Net-(D24-PadA): track 0.00 -> 13.6 mm
- net Net-(U4-Pad7): track 0.00 -> 3.31 mm
- net /GATE_BOTTOM: track 43.1 -> 40.2 mm
- net Net-(D25-PadA): vias 0 -> 6
- net Net-(D23-PadA): vias 0 -> 6
- added copper zone on B.Cu, net Net-(C12-Pad1)
- added copper zone on F.Cu, net Net-(C12-Pad1)
- added copper zone on B.Cu, net Net-(D23-PadA)
- added copper zone on F.Cu, net Net-(D23-PadA)
- added copper zone on B.Cu, net Net-(D25-PadA)
- added copper zone on F.Cu, net Net-(D25-PadA)
Other:
- board size 139.2 x 83.2 mm -> 139.2 x 105 mm

Commit message: placing back of bottom
Parts:
- removed C6: 100nF, Capacitor_SMD:C_0805_2012Metric
- removed D8: 1.5KE4A, Diode_THT:D_DO-201AD_P5.08mm_Vertical_AnodeUp
- removed F6: Fuse_Small, IGBT-DRIVER-emad:fuse.holder.1808
- removed R10: 2k/1w, Resistor_THT:R_Axial_DIN0414_L11.9mm_D4.5mm_P7.62mm_Vertical
- removed U5: ps2801, Package_SO:SOP-4_4.4x2.6mm_P1.27mm
- added C1: 100nF, Capacitor_SMD:C_1206_3216Metric_Pad1.33x1.80mm_HandSolder, F.Cu at (219.3, 164.8)
- added C2: 100nF, Capacitor_SMD:C_1206_3216Metric_Pad1.33x1.80mm_HandSolder, F.Cu at (221.7, 164.8)
- added D2: Dz4v, Diode_SMD:D_MELF, F.Cu at (138.2, 188.7)
- added D3: SMCJ7A, IGBT-DRIVER-emad:DIOM7959X250N, F.Cu at (231.0, 188.1)
- added G1: LOGO, IGBT-DRIVER-emad:koalaLogo, F.Cu at (120.0, 193.7)
- added R7: 6k, Resistor_SMD:R_1206_3216Metric, F.Cu at (115.3, 177.4)
- added R8: 6k, Resistor_SMD:R_1206_3216Metric, F.Cu at (115.3, 180.7)
- added R9: 6k, Resistor_SMD:R_1206_3216Metric, F.Cu at (120.9, 177.4)
- added Rex2: 1k, Resistor_SMD:R_0805_2012Metric, F.Cu at (159.7, 200.7)
- added U2: ps2801, Package_SO:SOP-4_4.4x2.6mm_P1.27mm, F.Cu at (153.6, 200.2)
- Cex3, D15, Qclamp2, Rex1, U1: moved to F.Cu
- Cex4, Cex5, Cex6, D14, Dex10, Q10, Q11, R23, Rex11, Rex12, Rex13, Rex14, Rex9: moved to B.Cu
- moved Cex5 54.7 mm to (210.9, 227.0)
- moved Q18 54.1 mm to (202.0, 226.3), turned to 0 degrees
- moved R16 53.2 mm to (209.1, 219.6), turned to 0 degrees
- moved R18 51.3 mm to (213.5, 224.1), turned to 0 degrees
- moved Rex14 51.0 mm to (212.7, 210.7), turned to 0 degrees
- moved R19 50.8 mm to (209.1, 222.5), turned to 0 degrees
- moved R6 46.5 mm to (203.9, 216.5), turned to 0 degrees
- moved Dex6 44.9 mm to (187.9, 226.3)
- moved C15 44.0 mm to (194.9, 222.6), turned to 0 degrees
- moved Rex12 43.2 mm to (208.3, 213.7), turned to 0 degrees
- moved Rex11 42.6 mm to (203.9, 210.4), turned to 0 degrees
- moved Q17 42.0 mm to (199.5, 217.2), turned to 0 degrees
- moved Rex15 41.4 mm to (212.7, 213.7), turned to 0 degrees
- moved Cex7 39.8 mm to (204.6, 219.5)
- moved D14 38.7 mm to (195.9, 226.4), turned to 0 degrees
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Connections:
- net /On_BOTTOM renamed /Gate Driver bottom/ItsOn
- net Net-(R12-Pad1) renamed /Gate Driver bottom/~Pulse-Disable
- C15 pad 2: GNDPWR -> /GND_BOTTOM
- D9 pad 1: GNDPWR -> (no net)
- Dex3 pad 2: Net-(Dex3-Pad2) -> /GATE_BOTTOM
- Dex4 pad 1: Net-(Dex3-Pad2) -> /GATE_BOTTOM
- Q12 pad 2: GNDPWR -> /GND_BOTTOM
- Q18 pad 2: GNDPWR -> /GND_BOTTOM
- R17 pad 2: /GATE_BOTTOM -> Net-(D3-PadA)
- R18 pad 2: GNDPWR -> /GND_BOTTOM
- Rex8 pad 2: /Gate Driver bottom/Vpp -> /VCC_BOTTOM
- Roff2 pad 1: Net-(Dex3-Pad2) -> /GATE_BOTTOM
- Roff4 pad 1: Net-(Dex3-Pad2) -> /GATE_BOTTOM
- Ron2 pad 2: Net-(Dex3-Pad2) -> /GATE_BOTTOM
- Ron3 pad 2: Net-(Dex3-Pad2) -> /GATE_BOTTOM
- U4 pad 7: Net-(U4-Pad7) -> (no net)
Routing:
- net /GND_BOTTOM: track 14.4 -> 174.8 mm, vias 0 -> 15
- net /Gate Driver bottom/Vpp: track 0.00 -> 89.6 mm, vias 0 -> 3
- net /EMITTER_BOTTOM: track 28.9 -> 103.7 mm, vias 0 -> 5
- net Net-(Rex9-Pad2): track 0.00 -> 45.1 mm, vias 0 -> 2
- net /VCC_BOTTOM: track 0.00 -> 36.3 mm
- net /Gate Driver bottom/ItsOn: track 0.00 -> 33.8 mm, vias 0 -> 1
- net Net-(C12-Pad2): track 0.26 -> 32.2 mm
- net /GATE_BOTTOM: track 40.2 -> 66.4 mm, vias 0 -> 1
- net Net-(Q20-Pad3): track 0.00 -> 13.8 mm
- net /Gate Driver bottom/on: track 0.00 -> 13.5 mm
- net /Gate Driver bottom/Control: track 0.00 -> 13.0 mm, vias 0 -> 1
- net Net-(C12-Pad1): track 0.00 -> 10.1 mm
- net Net-(Q19-Pad3): track 0.00 -> 8.00 mm
- net Net-(Cex4-Pad2): track 0.00 -> 7.67 mm
- net Net-(Q14-Pad2): track 0.00 -> 7.44 mm
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- added copper zone on B.Cu, net /GND_BOTTOM
- added copper zone on F.Cu, net /GND_BOTTOM
- added copper zone on F.Cu, net /Gate Driver bottom/Vpp
Other:
- board size 139.2 x 105 mm -> 139.2 x 93.5 mm
- board text added: "just a little more coOling !"

Commit message: a
Parts:
- D14, Rex13: moved to F.Cu
- moved R18 57.4 mm to (179.7, 177.6), turned to 90 degrees
- moved R19 52.3 mm to (182.3, 177.6), turned to 270 degrees
- moved R16 52.1 mm to (173.9, 181.1), turned to 270 degrees
- moved Q18 49.5 mm to (174.8, 184.9), turned to 180 degrees
- moved Dex6 47.5 mm to (206.0, 182.3), turned to 90 degrees
- moved R6 47.5 mm to (175.4, 178.4), turned to 180 degrees
- moved Cex5 42.3 mm to (199.0, 186.5)
- moved C15 41.5 mm to (179.5, 184.1)
- moved D14 39.7 mm to (189.4, 187.2), turned to 180 degrees
- moved Q10 39.2 mm to (202.0, 180.2), turned to 270 degrees
- moved Rex13 38.1 mm to (197.2, 186.6)
- moved D22 37.3 mm to (178.4, 181.2), turned to 180 degrees
- moved Cex7 35.7 mm to (203.8, 183.7), turned to 270 degrees
- moved Q17 35.6 mm to (180.5, 187.1)
- moved Dex7 35.3 mm to (174.7, 189.0), turned to 180 degrees
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Routing:
- net /GND_BOTTOM: track 174.8 -> 248.3 mm, vias 15 -> 16
- net /Gate Driver bottom/ItsOn: track 33.8 -> 99.2 mm, vias 1 -> 2
- net /Gate Driver bottom/fault: track 0.00 -> 54.4 mm, vias 0 -> 1
- net /Gate Driver bottom/Vpp: track 89.6 -> 138.5 mm, vias 3 -> 5
- net /Gate Driver bottom/Protection: track 0.00 -> 42.5 mm, vias 0 -> 2
- net /EMITTER_BOTTOM: track 103.7 -> 127.5 mm
- net /Gate Driver bottom/Collector: track 7.41 -> 26.4 mm
- net Net-(D14-Pad1): track 0.00 -> 15.4 mm, vias 0 -> 1
- net Net-(C15-Pad1): track 0.00 -> 9.73 mm
- net Net-(Cex5-Pad2): track 0.00 -> 8.66 mm
- net Net-(Dex7-Pad2): track 0.00 -> 7.41 mm
- net Net-(Cex4-Pad2): track 7.67 -> 14.6 mm
- net Net-(Cex7-Pad2): track 0.00 -> 6.27 mm
- net Net-(Rex9-Pad2): track 45.1 -> 51.3 mm, vias 2 -> 1
- net /Gate Driver bottom/on: track 13.5 -> 17.9 mm
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