File: IGBT DRIVER.kicad_pcb (KiCad board)
At the start: 2 copper layers, 139.2 x 93.5 mm, 131 parts, among them J1 Conn_02x05_Odd_Even, J3 Screw_Terminal_01x01, J5 Screw_Terminal_01x01, J6 Conn_01x02, J7 Conn_01x02, Q10 BC817, Q11 BC817, Q12 BC817, Q13 BC817, Q14 BC807, Q15 BC817, Q16 BC817, Q17 BC807, Q18 BC817, Q19 d44vh10, Q20 D45VH10, U1 ps2801, U2 ps2801, U4 6N136S, U6 ps2801, U7 miw06-24s24, U8 miw06-24s24

Commit message: added top parts
Parts:
- removed the C16 at (134.1, 170.0)
- removed the C4 at (122.5, 135.5)
- removed the D14 at (189.4, 187.2)
- removed the D9 at (122.4, 151.0)
- removed L2: 10uh, Inductor_SMD:L_12x12mm_H6mm
- removed Qclamp2: BUK7880-55A, Package_TO_SOT_SMD:SOT-223-3_TabPin2
- removed the R23 at (145.0, 197.0)
- removed the R3 at (123.9, 147.3)
- removed Rex1: 1k, Resistor_SMD:R_0805_2012Metric
- removed Rex10: 56k, Resistor_SMD:R_0805_2012Metric
- added BR1: DB107S, kicadFP:DIOB_DB107S, F.Cu at (121.9, 151.4)
- added C22: 1uF, Capacitor_SMD:C_1206_3216Metric_Pad1.33x1.80mm_HandSolder, F.Cu at (183.1, 173.9)
- added C3: 1uF, Capacitor_SMD:C_1206_3216Metric_Pad1.33x1.80mm_HandSolder, F.Cu at (218.2, 72.3)
- added C42: 1uF, Capacitor_SMD:C_1206_3216Metric_Pad1.33x1.80mm_HandSolder, F.Cu at (245.6, 44.5)
- added C43: 1uF, Capacitor_SMD:C_1206_3216Metric_Pad1.33x1.80mm_HandSolder, F.Cu at (221.4, 69.0)
- added C44: 1uF, Capacitor_SMD:C_1206_3216Metric_Pad1.33x1.80mm_HandSolder, F.Cu at (212.2, 78.7)
- added C45: 1uF, Capacitor_SMD:C_1206_3216Metric_Pad1.33x1.80mm_HandSolder, F.Cu at (225.6, 64.3)
- added C46: 1uF, Capacitor_SMD:C_1206_3216Metric_Pad1.33x1.80mm_HandSolder, F.Cu at (250.3, 41.1)
- added C47: 1uF, Capacitor_SMD:C_1206_3216Metric_Pad1.33x1.80mm_HandSolder, F.Cu at (239.6, 49.0)
- added C48: 1uF, Capacitor_SMD:C_1206_3216Metric_Pad1.33x1.80mm_HandSolder, F.Cu at (225.6, 61.0)
- added C49: 1uF, Capacitor_SMD:C_1206_3216Metric_Pad1.33x1.80mm_HandSolder, F.Cu at (203.5, 83.2)
- added C5: 1uF, Capacitor_SMD:C_1206_3216Metric_Pad1.33x1.80mm_HandSolder, F.Cu at (237.8, 54.1)
- added C51: 1uF, Capacitor_SMD:C_1206_3216Metric_Pad1.33x1.80mm_HandSolder, F.Cu at (231.7, 54.1)
- added C52: 1uF, Capacitor_SMD:C_1206_3216Metric_Pad1.33x1.80mm_HandSolder, F.Cu at (232.3, 57.5)
- added C53: 1uF, Capacitor_SMD:C_1206_3216Metric_Pad1.33x1.80mm_HandSolder, F.Cu at (215.4, 69.0)
- added C54: 1uF, Capacitor_SMD:C_1206_3216Metric_Pad1.33x1.80mm_HandSolder, F.Cu at (239.6, 45.6)
- added C55: 1uF, Capacitor_SMD:C_1206_3216Metric_Pad1.33x1.80mm_HandSolder, F.Cu at (204.3, 79.9)
- added C56: 96pF, Capacitor_SMD:C_0805_2012Metric, F.Cu at (247.4, 52.2)
- added C57: 100nF 250v, Capacitor_THT:C_Rect_L13.0mm_W4.0mm_P10.00mm_FKS3_FKP3_MKS4, F.Cu at (174.4, 42.2)
- added C58: 1uF, Capacitor_SMD:C_1206_3216Metric_Pad1.33x1.80mm_HandSolder, F.Cu at (219.6, 62.3)
- added C59: 1uF, Capacitor_SMD:C_1206_3216Metric_Pad1.33x1.80mm_HandSolder, F.Cu at (244.3, 41.1)
- added C60: 100nF, Capacitor_SMD:C_1206_3216Metric_Pad1.33x1.80mm_HandSolder, F.Cu at (221.6, 156.5)
- added C61: 100nF, Capacitor_SMD:C_1206_3216Metric_Pad1.33x1.80mm_HandSolder, F.Cu at (219.2, 156.5)
- added C62: 100pF, Capacitor_SMD:C_0805_2012Metric, F.Cu at (225.9, 45.1)
- added C63: 100pF, Capacitor_SMD:C_0805_2012Metric, F.Cu at (227.9, 71.2)
- added C64: 1nF, Capacitor_SMD:C_0805_2012Metric, F.Cu at (236.0, 61.9)
- added C65: 22nF, Capacitor_SMD:C_0805_2012Metric, F.Cu at (231.1, 68.2)
- added C66: 1nF, Capacitor_SMD:C_1206_3216Metric_Pad1.33x1.80mm_HandSolder, F.Cu at (219.6, 65.6)
- added C67: 10nF, Capacitor_SMD:C_0805_2012Metric, F.Cu at (226.7, 67.5)
- added C68: C, Capacitor_SMD:C_0805_2012Metric, F.Cu at (215.0, 150.0)
- added D12: 1n4148, Diode_SMD:D_SMA, B.Cu at (164.1, 186.1)
- added D16: Dz10v, Diode_SMD:D_MELF, F.Cu at (189.4, 187.2)
- added D2: LED_Green_0805, kicadFP:GREEN_LED_0805, B.Cu at (126.5, 190.4)
- added D23: LED_Blue_0805, kicadFP:LED_BLUE_0805, F.Cu at (168.4, 197.2)
- added D24: Dz4v, Diode_SMD:D_MELF, F.Cu at (232.7, 50.4)
- added D25: SMCJ160CA-13-F, IGBT-DRIVER-emad:DIOM7959X250N, F.Cu at (190.5, 67.9)
- added D26: SMCJ160CA-13-F, IGBT-DRIVER-emad:DIOM7959X250N, F.Cu at (218.4, 43.2)
- added D27: SMCJ160CA-13-F, IGBT-DRIVER-emad:DIOM7959X250N, F.Cu at (178.4, 77.6)
- added D28: SMCJ160CA-13-F, IGBT-DRIVER-emad:DIOM7959X250N, F.Cu at (205.5, 51.2)
- added D3: SMCJ160CA-13-F, IGBT-DRIVER-emad:DIOM7959X250N, F.Cu at (203.2, 60.5)
- added D30: SMCJ160CA-13-F, IGBT-DRIVER-emad:DIOM7959X250N, F.Cu at (191.7, 60.5)
- added D31: 1n4148, Diode_SMD:D_SMA, F.Cu at (224.7, 49.1)
- added D32: SMCJ7A, IGBT-DRIVER-emad:DIOM7959X250N, F.Cu at (178.4, 70.2)
- added D33: 26v Zener, Diode_SMD:D_MELF, F.Cu at (232.7, 46.1)
- added D34: LED_RED_0805, kicadFP:LED_RED_0805_2012Metric, F.Cu at (243.0, 56.7)
- added D35: BYV26E, Diode_THT:D_DO-35_SOD27_P7.62mm_Horizontal, F.Cu at (173.7, 83.1)
- added D36: Dz10v, Diode_SMD:D_MELF, F.Cu at (208.5, 71.5)
- added D37: LED_Blue_0805, kicadFP:LED_BLUE_0805, F.Cu at (249.3, 48.8)
- added D38: 1n4148, Diode_SMD:D_SMA, F.Cu at (237.3, 41.7)
- added D39: 1n4148, Diode_SMD:D_SMA, F.Cu at (224.7, 53.7)
- added D40: BZX85C20, Diode_SMD:D_MELF, F.Cu at (208.5, 67.3)
- added D41: 1n4148, Diode_SMD:D_SMA, F.Cu at (196.4, 82.2)
- added D42: 1n4148, Diode_SMD:D_SMA, F.Cu at (197.3, 76.2)
- added D43: 1n4148, Diode_SMD:D_SMA, F.Cu at (212.6, 62.9)
- added F3: Fuse, IGBT-DRIVER-emad:fuse.holder.1808, F.Cu at (178.0, 45.7)
- added L1: 10uh, kicadFP:L_12x12mm_H6mm, F.Cu at (122.4, 167.1)
- added LOGO1: Logo_Open_Hardware_Small, Symbol:OSHW-Logo_5.7x6mm_SilkScreen, F.Cu at (115.3, 202.9)
- added Q13: BC817, Package_TO_SOT_SMD:SOT-23, F.Cu at (209.6, 82.6)
- added Q14: BC807, Package_TO_SOT_SMD:SOT-23, F.Cu at (214.0, 82.6)
- added Q15: BC817, Package_TO_SOT_SMD:SOT-23, F.Cu at (237.5, 58.1)
- added Q16: BC817, Package_TO_SOT_SMD:SOT-23, F.Cu at (250.8, 45.0)
- added Q17: BC817, Package_TO_SOT_SMD:SOT-23, F.Cu at (243.0, 53.0)
- added Q18: BUK7880-55A, Package_TO_SOT_SMD:SOT-223-3_TabPin2, F.Cu at (227.3, 139.5)
- added Q19: BC817, Package_TO_SOT_SMD:SOT-23, F.Cu at (223.4, 72.9)
- added Q20: BC817, Package_TO_SOT_SMD:SOT-23, F.Cu at (217.4, 76.3)
- added Q21: BC807, Package_TO_SOT_SMD:SOT-23, F.Cu at (244.8, 48.4)
- added Q22: BC817, Package_TO_SOT_SMD:SOT-23, F.Cu at (231.5, 61.5)
- added Q23: d44vh10, Package_TO_SOT_SMD:TO-252-2, F.Cu at (196.6, 140.3)
- added Q24: D45VH10, Package_TO_SOT_SMD:TO-252-2, F.Cu at (196.6, 152.9)
- added Q6: BUK7880-55A, Package_TO_SOT_SMD:SOT-223-3_TabPin2, F.Cu at (227.0, 180.1)
- added R10: 1k, Resistor_SMD:R_0805_2012Metric, F.Cu at (146.5, 197.7)
- added R13: 1k, Resistor_SMD:R_0805_2012Metric, F.Cu at (159.9, 200.4)
- added R22: 56k, Resistor_SMD:R_0805_2012Metric, B.Cu at (193.6, 172.5)
- added R37: 20K, Resistor_SMD:R_0805_2012Metric, F.Cu at (213.0, 170.7)
- added R39: 220, Resistor_SMD:R_0805_2012Metric, F.Cu at (168.4, 193.6)
- added R40: 1k, Resistor_SMD:R_0805_2012Metric, F.Cu at (164.8, 193.5)
- added R41: 1k, Resistor_SMD:R_0805_2012Metric, F.Cu at (247.4, 55.2)
- added R42: 6.8k, Resistor_SMD:R_0805_2012Metric, F.Cu at (232.3, 71.2)
- added R43: 20K, Resistor_THT:R_Axial_DIN0207_L6.3mm_D2.5mm_P10.16mm_Horizontal, F.Cu at (173.7, 56.4)
- added R44: 1k, Resistor_SMD:R_0805_2012Metric, F.Cu at (222.8, 79.6)
- added R45: 1k, Resistor_SMD:R_0805_2012Metric, F.Cu at (235.5, 68.2)
- added R46: 220, Resistor_THT:R_Axial_DIN0207_L6.3mm_D2.5mm_P10.16mm_Horizontal, F.Cu at (188.3, 41.5)
- added R47: 120, Resistor_SMD:R_0805_2012Metric, F.Cu at (240.4, 61.9)
- added R48: 2.2k, Resistor_SMD:R_0805_2012Metric, F.Cu at (227.8, 74.2)
- added R49: 2.2k, Resistor_SMD:R_0805_2012Metric, F.Cu at (218.4, 83.0)
- added R50: 1k, Resistor_SMD:R_0805_2012Metric, F.Cu at (235.5, 65.2)
- added R51: 220, Resistor_SMD:R_0805_2012Metric, F.Cu at (239.9, 64.9)
- added R52: 220, Resistor_SMD:R_0805_2012Metric, F.Cu at (221.8, 76.7)
- added R53: 3.3K, Resistor_SMD:R_0805_2012Metric, F.Cu at (247.4, 58.1)
- added R54: 1k, Resistor_SMD:R_0805_2012Metric, F.Cu at (227.2, 83.1)
- added R55: 56k, Resistor_SMD:R_0805_2012Metric, F.Cu at (236.7, 74.2)
- added R56: 1k, Resistor_SMD:R_0805_2012Metric, F.Cu at (251.8, 57.7)
- added R57: 2.2k, Resistor_SMD:R_0805_2012Metric, F.Cu at (231.7, 77.2)
- added R58: 2.2k, Resistor_SMD:R_0805_2012Metric, F.Cu at (244.3, 64.8)
- added R59: 1.5k, Resistor_SMD:R_0805_2012Metric, F.Cu at (236.7, 71.1)
- added R60: 1.8k, Resistor_SMD:R_0805_2012Metric, F.Cu at (251.9, 54.8)
- added R61: 1K, Resistor_SMD:R_0805_2012Metric, F.Cu at (227.2, 80.1)
- added R62: 1K, Resistor_SMD:R_0805_2012Metric, F.Cu at (239.9, 67.8)
- added R63: 1k, Resistor_SMD:R_0805_2012Metric, F.Cu at (227.2, 77.2)
- added R64: 1K, Resistor_SMD:R_0805_2012Metric, F.Cu at (244.8, 61.1)
- added R65: 10, Resistor_SMD:R_0805_2012Metric, F.Cu at (232.2, 74.2)
- added R66: 40, Resistor_SMD:R_2512_6332Metric, F.Cu at (200.2, 66.6)
- added R67: 40, Resistor_SMD:R_2512_6332Metric, F.Cu at (212.9, 58.2)
- added R68: 40, Resistor_SMD:R_2512_6332Metric, F.Cu at (200.2, 71.5)
- added R69: 40, Resistor_SMD:R_2512_6332Metric, F.Cu at (188.1, 82.4)
- added R70: 20K, Resistor_SMD:R_0805_2012Metric, F.Cu at (217.0, 150.0)
- added R71: 20K, Resistor_SMD:R_0805_2012Metric, F.Cu at (213.0, 150.0)
- added R8: 1k, Resistor_SMD:R_0805_2012Metric, F.Cu at (251.9, 51.8)
- added U10: ps2801, Package_SO:SOP-4_4.4x2.6mm_P1.27mm, F.Cu at (188.5, 77.8)
- added U7: 6N136S, Package_DIP:SMDIP-8_W9.53mm, F.Cu at (192.7, 50.9)
- added U8: ps2801, Package_SO:SOP-4_4.4x2.6mm_P1.27mm, F.Cu at (188.5, 73.7)
- added U9: ps2801, Package_SO:SOP-4_4.4x2.6mm_P1.27mm, F.Cu at (228.5, 41.5)
- C4: renamed from C17; moved to B.Cu
- C6: renamed from C9; moved to B.Cu
- D1: value LED -> LED_RED_0805; footprint LED_SMD:LED_1206_3216Metric_Castellated -> kicadFP:LED_RED_0805_2012Metric
- D29: value DF10M -> Dz8v; footprint Diode_SMD:Diode_Bridge_Vishay_DFS -> Diode_SMD:D_MELF
- R1: renamed from R7; moved to B.Cu
- R2: renamed from R8; moved to B.Cu
- R38: renamed from R21; value 10K -> 20K
- R4: renamed from R9; moved to B.Cu
- R7: renamed from R1; moved to B.Cu
- moved D29 124.9 mm to (205.2, 76.1)
- moved C50 102.7 mm to (212.2, 75.3), turned to 0 degrees
- moved D1 71.0 mm to (164.8, 197.3), turned to 90 degrees
- moved R2 59.8 mm to (164.0, 146.0)
- moved R1 59.3 mm to (164.0, 143.5)
- moved F1 58.6 mm to (127.3, 133.3), turned to 270 degrees
- moved C10 56.7 mm to (172.0, 134.5)
- moved R4 51.8 mm to (164.0, 148.6)
- moved C9 49.4 mm to (171.8, 130.4)
- moved C1 41.0 mm to (134.9, 172.2), turned to 270 degrees
- moved R7 37.5 mm to (125.8, 187.5), turned to 90 degrees
- moved C4 36.2 mm to (144.9, 173.4), turned to 90 degrees
- moved C6 35.8 mm to (144.8, 147.6), turned to 90 degrees
- moved J2 25.5 mm to (195.2, 126.3)
- moved C2 2.94 mm to (134.9, 146.6), turned to 270 degrees
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- renumbered C8 to C1, C20 to C10, C13 to C12, C41 to C13, C42 to C14, C43 to C15, C44 to C16, C45 to C17, C46 to C18, C47 to C19, C3 to C2, C48 to C20, C49 to C21, C51 to C23, C52 to C24, C53 to C25, C54 to C26, C55 to C27, C56 to C28, Cex3 to C29, C12 to C30, C57 to C31, C58 to C32, C1 to C33, C2 to C34, Cex4 to C35, Cex5 to C36, Cex6 to C37, Cex7 to C38, C15 to C39, C14 to C40, Cclamp2 to C41, C18 to C7, C7 to C8, C19 to C9, D28 to D11, D3 to D13, D15 to D14, D13 to D15, Dex6 to D17, Dex7 to D18, D22 to D19, Dex10 to D20, Dex3 to D21, Dex4 to D22, D23 to D4, D2 to D5, D24 to D6, D25 to D7, D26 to D8, D27 to D9, F4 to F2, H2 to H1, H3 to H2, H1 to H3, J3 to J2, J5 to J3, J6 to J4, J7 to J5, Q10 to Q1, Q15 to Q10, Q19 to Q11, Q20 to Q12, Q17 to Q2, Q11 to Q3, Q12 to Q4, Q18 to Q5, Q13 to Q7, Q16 to Q8, Q14 to Q9, Rex8 to R11, R14 to R12, Rex2 to R14, R17 to R15, Rex9 to R16, Rex11 to R17, Rex12 to R18, Rex13 to R19, R13 to R20, Rex14 to R21, Rex15 to R23, Rex16 to R24, Rex17 to R25, R6 to R26, R16 to R27, R18 to R28, R19 to R29, R4 to R3, Rex18 to R30, R22 to R31, R15 to R32, Ron3 to R33, Roff4 to R34, Ron2 to R35, Roff2 to R36, R2 to R5, R5 to R6, R12 to R9, U8 to U1, U7 to U2, U4 to U3, U1 to U4, U6 to U5, U2 to U6
Connections:
- net /Gate Driver bottom/~Pulse-Disable renamed /On_TOP
- C50 pad 1: /GND_BOTTOM -> /GND_top
- C50 pad 2: /EMITTER_BOTTOM -> /sheet61D91DB7/Vpp
- D1 pad 1: GNDD -> /Gate Driver bottom/fault
- D29 pad 1: /Vin- -> /EMITTER_TOP
- D29 pad 2: Net-(D29-Pad2) -> /GND_top
- F1 pad 2: Net-(D29-Pad2) -> Net-(BR1-PadAC1)
- J1 pad 2: (no net) -> /Reset_top
- J1 pad 4: (no net) -> /Pulse-TOP
- J1 pad 8: (no net) -> /Error_top
- J2 pad 1: Net-(J3-Pad1) -> /sheet61D91DB7/Collector
- J4 pad 1: (no net) -> /GATE_TOP
- J4 pad 2: (no net) -> /EMITTER_TOP
- R7 pad 1: Net-(D1-Pad2) -> Net-(D2-Pad2)
- U3 pad 3: /Vin- -> GNDD
- U3 pad 7: (no net) -> Net-(D12-Pad2)
- U4 pad 2: /GND_BOTTOM -> /Gate Driver bottom/fault
- U4 pad 3: /Vin- -> GNDD
- U6 pad 3: /Vin- -> GNDD
- U6 pad 4: (no net) -> /ON_Bottom
Routing:
- net +15V: track 0.00 -> 116.8 mm
- net GNDD: track 0.00 -> 102.4 mm
- net /Error_BOTTOM: track 0.00 -> 86.8 mm, vias 0 -> 1
- net /Reset_BOTTOM: track 0.00 -> 71.5 mm
- net /Vin+: track 0.00 -> 50.3 mm
- net /Pulse-BOTTOM: track 0.00 -> 50.0 mm
- net /Gate Driver bottom/Vpp: track 138.5 -> 164.6 mm, vias 5 -> 6
- net /Vin-: track 0.00 -> 22.6 mm
- net /Gate Driver bottom/fault: track 54.4 -> 76.1 mm, vias 1 -> 2
- net /GND_BOTTOM: track 248.3 -> 261.6 mm, vias 16 -> 23
- net Net-(BR1-PadAC1): track 0.00 -> 8.87 mm
- net Net-(BR1-Pad+): track 0.00 -> 7.94 mm
- net Net-(D12-Pad2): track 0.00 -> 6.13 mm, vias 0 -> 1
- net /On_TOP: track 0.00 -> 4.24 mm
- net Net-(R10-Pad1): track 0.00 -> 4.07 mm
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Other:
- outline, holes or cut-outs redrawn
- board text added: "E"
- board text added: "Fault"
- board text added: "G"
- board text added: "Power"
- board text added: "VERY HIGH VOLTAGE !"
- board text added: "VERY HIGH VOLTAGE!"

Commit message: topside added
Parts:
- added D44: LED_RED_0805, kicadFP:LED_RED_0805, F.Cu at (115.9, 136.6)
- added R72: 1.8k, Resistor_SMD:R_0805_2012Metric, B.Cu at (126.6, 186.5)
- added R73: 1.8k, Resistor_SMD:R_0805_2012Metric, B.Cu at (122.7, 186.5)
- added R74: 1.8k, Resistor_SMD:R_0805_2012Metric, F.Cu at (116.0, 132.5)
- C62, C63, C64, C65, C66, C67, D27, D28, D29, D3, D31, D38, D39, D40, Q13, Q14, Q15, Q16, Q17, Q19, Q20, Q21, Q22, R42, R47, R48, R49, R51, R53, R54, R55, R56, R57, R58, R59, R60, R61, R62, R63, R64, R65: moved to B.Cu
- D1, D34: footprint kicadFP:LED_RED_0805_2012Metric -> kicadFP:LED_RED_0805
- D2: footprint kicadFP:GREEN_LED_0805 -> Diode_SMD:D_0805_2012Metric; moved to F.Cu
- D24, D5: value Dz4v -> LED_Yellow_0805; footprint Diode_SMD:D_MELF -> kicadFP:LED_Yellow_0805; moved to B.Cu
- R7: moved to F.Cu
- moved D24 177.9 mm to (122.7, 190.2), turned to 90 degrees
- moved R8 132.7 mm to (144.8, 130.3)
- moved R41 128.9 mm to (144.7, 132.9)
- moved C46 125.2 mm to (188.2, 149.7)
- moved C42 124.7 mm to (188.2, 155.2)
- moved C56 117.4 mm to (161.7, 132.4), turned to 90 degrees
- moved C5 117.3 mm to (183.1, 158.0), turned to 180 degrees
- moved C47 115.5 mm to (183.1, 149.7), turned to 180 degrees
- moved Q16 114.0 mm to (196.1, 145.0)
- moved C59 113.0 mm to (183.1, 136.1), turned to 180 degrees
- moved R60 112.5 mm to (177.5, 139.2), turned to 90 degrees
- moved U9 112.0 mm to (153.5, 124.7)
- moved D37 111.1 mm to (167.9, 124.5), turned to 90 degrees
- moved C62 108.6 mm to (193.0, 148.5), turned to 90 degrees
- moved Q21 108.2 mm to (203.4, 148.3), turned to 90 degrees
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Connections:
- net /sheet61D91DB7/Collector renamed /Gate Driver top/Collector
- net /sheet61D91DB7/Control renamed /Gate Driver top/Control
- net /sheet61D91DB7/ItsOn renamed /Gate Driver top/ItsOn
- net /sheet61D91DB7/Protection renamed /Gate Driver top/Protection
- net /sheet61D91DB7/Vpp renamed /Gate Driver top/Vpp
- net /sheet61D91DB7/fault renamed /Gate Driver top/fault
- net /sheet61D91DB7/on renamed /Gate Driver top/on
- D24 pad 1: /Pulse-TOP -> GNDD
- D5 pad 1: /Pulse-BOTTOM -> GNDD
- J1 pad 6: /Vin+ -> (no net)
- J1 pad 9: (no net) -> /Vin+
- R16 pad 2: Net-(R16-Pad2) -> Net-(D12-Pad2)
- R47 pad 2: Net-(R47-Pad2) -> Net-(D31-Pad2)
- R8 pad 2: Net-(D24-Pad2) -> /Pulse-TOP
- R9 pad 2: Net-(D5-Pad2) -> /Pulse-BOTTOM
- U3 pad 6: Net-(R16-Pad2) -> Net-(D12-Pad2)
- U3 pad 7: Net-(D12-Pad2) -> (no net)
- U7 pad 6: Net-(R47-Pad2) -> Net-(D31-Pad2)
- U7 pad 7: Net-(D31-Pad2) -> (no net)
Routing:
- net /GND_top: track 0.00 -> 180.9 mm, vias 0 -> 16
- net /Gate Driver top/Vpp: track 0.00 -> 103.7 mm, vias 0 -> 4
- net /Gate Driver top/ItsOn: track 0.00 -> 94.1 mm, vias 0 -> 2
- net /GATE_TOP: track 0.00 -> 60.9 mm, vias 0 -> 2
- net Net-(D12-Pad2): track 6.13 -> 61.6 mm
- net Net-(R16-Pad2): track 51.3 -> 0.00 mm, vias 1 -> 0
- net /Pulse-TOP: track 0.00 -> 51.1 mm, vias 0 -> 1
- net /VCC_top: track 0.00 -> 49.1 mm
- net /Gate Driver top/fault: track 0.00 -> 45.1 mm
- net /EMITTER_TOP: track 0.00 -> 44.5 mm, vias 0 -> 1
- net /Gate Driver top/Protection: track 0.00 -> 38.5 mm, vias 0 -> 1
- net GNDD: track 102.4 -> 140.2 mm, vias 0 -> 2
- net Net-(D31-Pad2): track 0.00 -> 34.4 mm
- net Net-(D41-Pad2): track 0.00 -> 27.9 mm, vias 0 -> 1
- net /Gate Driver top/on: track 0.00 -> 26.1 mm
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- added copper zone on B.Cu, net /GND_top
- added copper zone on F.Cu, net /GND_top
- added copper zone on F.Cu, net /Gate Driver top/Vpp
- added copper zone on B.Cu, net Net-(C57-Pad1)
- added copper zone on F.Cu, net Net-(C57-Pad1)
- added copper zone on B.Cu, net Net-(D25-PadC)
- added copper zone on F.Cu, net Net-(D25-PadC)
- added copper zone on B.Cu, net Net-(D26-PadA)
- added copper zone on F.Cu, net Net-(D26-PadA)
Other:
- board size 139.2 x 93.5 mm -> 139.2 x 95.6 mm
- board text added: "Fuse"
- board text added: "PNP gets hot in faults"

Commit message: yii
Parts:
- D2: footprint Diode_SMD:D_0805_2012Metric -> kicadFP:LED_Green_0805
- moved R41 10.8 mm to (146.3, 122.2), turned to 90 degrees
- moved C56 3.21 mm to (161.6, 129.2)
- moved R8 0.53 mm to (144.6, 130.8), turned to 180 degrees
- moved D2 0.09 mm to (127.5, 136.0)
Routing:
- net /Reset_top: track 0.00 -> 111.3 mm, vias 0 -> 3
- net GNDD: track 140.2 -> 238.6 mm, vias 2 -> 4
- net /Error_top: track 0.00 -> 82.8 mm, vias 0 -> 1
- net /Pulse-TOP: track 51.1 -> 132.3 mm
- net /EMITTER_TOP: track 44.5 -> 115.6 mm, vias 1 -> 2
- net /GND_top: track 180.9 -> 216.6 mm, vias 16 -> 21
- net /Gate Driver top/Vpp: track 103.7 -> 125.2 mm
- net /Gate Driver top/fault: track 45.1 -> 54.8 mm, vias 0 -> 2
- net /Gate Driver top/Protection: track 38.5 -> 43.6 mm, vias 1 -> 2
- net Net-(D31-Pad2): track 34.4 -> 39.2 mm, vias 0 -> 1
- net Net-(R41-Pad1): track 0.00 -> 4.70 mm
- net Net-(R44-Pad1): track 0.00 -> 4.58 mm
- net /Error_BOTTOM: track 86.8 -> 83.0 mm
- net /ON_Bottom: track 0.00 -> 3.66 mm
- net +15V: track 125.8 -> 123.4 mm
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- added copper zone on B.Cu, net (none)
- added copper zone on F.Cu, net (none)
Other:
- board text added: "EB"
- board text added: "ET"
- board text added: "P T"
- board text added: "PB"
- board text added: "PT"
- board text added: "RB"
- board text added: "V+"
- board text added: "V-"
