File: IGBT DRIVER.kicad_pcb (KiCad board)
At the start: 2 copper layers, 139.2 x 95.6 mm, 240 parts, among them J1 Conn_02x05_Odd_Even, J2 Screw_Terminal_01x01, J3 Screw_Terminal_01x01, J4 Conn_01x02, J5 Conn_01x02, Q1 BC817, Q10 BC817, Q11 d44vh10, Q12 D45VH10, Q13 BC817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

Commit message: add some wiki pics
Parts:
- J1: footprint Connector_IDC:IDC-Header_2x05-1MP_P2.54mm_Latch_Horizontal -> kicadFP:IDC-Header_2x05-1MP_P2.54mm_Latch_Horizontal
Routing:
- net Net-(U3-Pad7): track 0.00 -> 0.59 mm
- net (no net): track 0.59 -> 0.00 mm
