File: IGBT DRIVER.sch (KiCad schematic (older format))
At the start: 28 parts, among them J1 Conn_01x04, J2 Conn_01x04, J3 Screw_Terminal_01x01, J4 Conn_01x04, J5 Screw_Terminal_01x01, U1 miw06-24s24

Commit message: skm200 3d
Parts:
- removed D12: 1.5KE4A, Diode_THT:D_DO-201AD_P5.08mm_Vertical_AnodeUp, symbol Diode:1.5KExxA
- removed D15: 1.5KE24A, Diode_THT:D_DO-201AD_P5.08mm_Vertical_AnodeUp, symbol Diode:1.5KExxA
- removed JP2: SolderJumper_2_Bridged, Jumper:SolderJumper-2_P1.3mm_Bridged_Pad1.0x1.5mm, symbol Jumper:SolderJumper_2_Bridged
- added C16, C18: 10uf/35v, Capacitor_THT:CP_Radial_D5.0mm_P2.50mm, symbol Device:CP
- added C17: 100nf, Capacitor_SMD:C_1206_3216Metric_Pad1.33x1.80mm_HandSolder, symbol Device:C
- added C19: 1uF, Capacitor_SMD:C_1206_3216Metric_Pad1.33x1.80mm_HandSolder, symbol Device:C
- added C20: 100nF, Capacitor_SMD:C_1206_3216Metric_Pad1.33x1.80mm_HandSolder, symbol Device:C
- added L1: 10uh, gh- kicad:INDUCTOR.SMD.12, symbol Device:L
- added R10: 2k/1w, Resistor_THT:R_Axial_DIN0414_L11.9mm_D4.5mm_P7.62mm_Vertical, symbol Device:R
- added U6: miw06-24s24, gh- kicad:MIWI06, symbol IGBT-DRIVER-rescue:miw06-24s24-GH-kicad
Connections:
- net labels removed: VPP
- wire segments 100 -> 121
Other:
- note removed: "cut jumper for -5v bias"
- moved on the sheet: C11, C13, C3, C4, C7, C9, L2, R4

Commit message: changed bjt
Parts:
- added H5: MountingHole, MountingHole:MountingHole_4.3x6.2mm_M4_Pad_Via, symbol Mechanical:MountingHole
- added IGBTSymbol1: SYM_Arrow45_Normal, IGBT-DRIVER-emad:skm200GB, symbol Graphic:SYM_Arrow45_Normal
- added J6, J7: Conn_01x02, IGBT-DRIVER-emad:IGBT_Socket, symbol Connector_Generic:Conn_01x02
- H1, H2, H3, H4: footprint TestPoint:TestPoint_Plated_Hole_D4.0mm -> MountingHole:MountingHole_4.3x6.2mm_M4_Pad_Via
Changed lines of the file:
@@
 F 0 "H4" H 5625 4466 50  0000 L CNN
 F 1 "MountingHole" H 5625 4375 50  0000 L CNN
-F 2 "TestPoint:TestPoint_Plated_Hole_D4.0mm" H 5525 4420 50  0001 C CNN
+F 2 "MountingHole:MountingHole_4.3x6.2mm_M4_Pad_Via" H 5525 4420 50  0001 C CNN
 F 3 "~" H 5525 4420 50  0001 C CNN
 	1    5525 4420
@@
 F 0 "H3" H 4830 4461 50  0000 L CNN
 F 1 "MountingHole" H 4830 4370 50  0000 L CNN
-F 2 "TestPoint:TestPoint_Plated_Hole_D4.0mm" H 4730 4415 50  0001 C CNN
+F 2 "MountingHole:MountingHole_4.3x6.2mm_M4_Pad_Via" H 4730 4415 50  0001 C CNN
 F 3 "~" H 4730 4415 50  0001 C CNN
 	1    4730 4415
@@
 F 0 "H2" H 4830 4226 50  0000 L CNN
 F 1 "MountingHole" H 4830 4135 50  0000 L CNN
-F 2 "TestPoint:TestPoint_Plated_Hole_D4.0mm" H 4730 4180 50  0001 C CNN
+F 2 "MountingHole:MountingHole_4.3x6.2mm_M4_Pad_Via" H 4730 4180 50  0001 C CNN
 F 3 "~" H 4730 4180 50  0001 C CNN
 	1    4730 4180
@@
 F 0 "H1" H 5620 4221 50  0000 L CNN
 F 1 "MountingHole" H 5620 4130 50  0000 L CNN
-F 2 "TestPoint:TestPoint_Plated_Hole_D4.0mm" H 5520 4175 50  0001 C CNN
+F 2 "MountingHole:MountingHole_4.3x6.2mm_M4_Pad_Via" H 5520 4175 50  0001 C CNN
 F 3 "~" H 5520 4175 50  0001 C CNN
 	1    5520 4175
@@
 Text Label 3855 6105 0    50   ~ 0
 GND_top
+$Comp
+L Connector_Generic:Conn_01x02 J6
+U 1 1 6199921A
+P 12125 3190
+F 0 "J6" H 12205 3182 50  0000 L CNN
+F 1 "Conn_01x02" H 12205 3091 50  0000 L CNN
+F 2 "IGBT-DRIVER-emad:IGBT_Socket" H 12125 3190 50  0001 C CNN
+F 3 "~" H 12125 3190 50  0001 C CNN
+	1    12125 3190
+	1    0    0    -1
+$EndComp
+Text Label 11925 3190 2    50   ~ 0
+GATE_TOP
+Text Label 11925 3290 2    50   ~ 0
+EMITTER_TOP
+$Comp
+L Connector_Generic:Conn_01x02 J7
+U 1 1 619998BE
+P 12715 6300
+F 0 "J7" H 12795 6292 50  0000 L CNN
+F 1 "Conn_01x02" H 12795 6201 50  0000 L CNN
+F 2 "IGBT-DRIVER-emad:IGBT_Socket" H 12715 6300 50  0001 C CNN
+F 3 "~" H 12715 6300 50  0001 C CNN
+	1    12715 6300
+	1    0    0    -1
+$EndComp
+Text Label 12515 6300 2    50   ~ 0
+GATE_BOTTOM
+Text Label 12515 6400 2    50   ~ 0
+EMITTER_BOTTOM
+$Comp
+L Graphic:SYM_Arrow45_Normal IGBTSymbol?
+U 1 1 619CFF89
+P 5455 2025
+AR Path="/6309618D/619CFF89" Ref="IGBTSymbol?"  Part="1"
+AR Path="/6340E1F3/619CFF89" Ref="IGBTSymbol?"  Part="1"
+AR Path="/619CFF89" Ref="IGBTSymbol1"  Part="1"
+F 0 "IGBTSymbol1" H 5605 2075 50  0000 C CNN
+F 1 "SYM_Arrow45_Normal" H 5455 1925 50  0001 C CNN
+F 2 "IGBT-DRIVER-emad:skm200GB" H 5455 2025 50  0001 C CNN
+F 3 "~" H 5455 2025 50  0001 C CNN
+	1    5455 2025
+	1    0    0    -1
+$EndComp
+$Comp
+L Mechanical:MountingHole H5
+U 1 1 61C062DA
+P 4240 4430
+F 0 "H5" H 4340 4476 50  0000 L CNN
+F 1 "MountingHole" H 4340 4385 50  0000 L CNN
+F 2 "MountingHole:MountingHole_4.3x6.2mm_M4_Pad_Via" H 4240 4430 50  0001 C CNN
+F 3 "~" H 4240 4430 50  0001 C CNN
+	1    4240 4430
+	1    0    0    -1
+$EndComp
 $EndSCHEMATC

Commit message: some placement
Parts:
- removed J1, J2, J4: Conn_01x04, gh- kicad:WJ250-3.5, symbol Connector_Generic:Conn_01x04
- removed L1: 10uh, gh- kicad:INDUCTOR.SMD.12, symbol Device:L
- added J1: Conn_02x05_Odd_Even, Connector_IDC:IDC-Header_2x05-1MP_P2.54mm_Latch_Horizontal, symbol Connector_Generic:Conn_02x05_Odd_Even
- F1: footprint gh- kicad:fuse.holder.1808 -> IGBT-DRIVER-emad:fuse.holder.1808
- J3, J5: footprint (none) -> IGBT-DRIVER-emad:COOLERI
- L2: footprint gh- kicad:INDUCTOR.SMD.12 -> Inductor_SMD:L_12x12mm_H6mm
- R1, R3: footprint Resistor_SMD:R_0805_2012Metric_Pad1.15x1.40mm_HandSolder -> Resistor_SMD:R_0805_2012Metric
- U1, U6: footprint gh- kicad:MIWI06 -> IGBT-DRIVER-emad:MIWI06
Connections:
- net labels removed: EMITTER_DOWN, Error, Fault-Reset, GATE_DOWN
- wire segments 121 -> 115
Other:
- moved on the sheet: D1, D9, IGBTSymbol1, L2, R1, R3

Commit message: some placements have done
Parts:
- removed U1, U6: miw06-24s24, IGBT-DRIVER-emad:MIWI06, symbol IGBT-DRIVER-rescue:miw06-24s24-GH-kicad
- added R2, R5: 6k, Resistor_SMD:R_1206_3216Metric, symbol Device:R
- added U7, U8: miw06-24s24, IGBT-DRIVER-emad:MIWI06, symbol GateDriver:miw06-24s24
- R4: value 2k/1w -> 6k; footprint Resistor_THT:R_Axial_DIN0414_L11.9mm_D4.5mm_P7.62mm_Vertical -> Resistor_SMD:R_1206_3216Metric
Connections:
- wire segments 115 -> 123
- no-connect marks 0 -> 2
Other:
- moved on the sheet: C11, C13, C7
Changed lines of the file:
@@
 EESchema Schematic File Version 4
-LIBS:IGBT DRIVER-cache
-EELAYER 29 0
+EELAYER 30 0
 EELAYER END
 $Descr A3 16535 11693
 encoding utf-8
-Sheet 1 3
+Sheet 1 2
 Title ""
 Date ""
@@
 Connection ~ 1885 1135
 Wire Wire Line
-	3790 1615 3790 1575
-Wire Wire Line
-	3790 1195 3790 1275
-Wire Wire Line
-	3475 1555 3475 1615
-Connection ~ 3475 1615
-Wire Wire Line
-	3475 1615 3790 1615
-Wire Wire Line
-	3475 1195 3475 1255
-Wire Wire Line
-	3305 1195 3475 1195
-Connection ~ 3475 1195
+	4170 1615 4170 1575
+Wire Wire Line
+	4170 1195 4170 1275
 $Comp
 L power:+15V #PWR03
@@
 Connection ~ 1455 1685
 Wire Wire Line
-	4520 1195 4520 1265
-Wire Wire Line
-	4520 1565 4520 1615
-Wire Wire Line
-	4520 1615 4235 1615
-Wire Wire Line
-	4235 1565 4235 1615
-Wire Wire Line
-	4235 1195 4520 1195
-Wire Wire Line
-	4235 1195 4235 1265
+	4900 1195 4900 1265
+Wire Wire Line
+	4900 1565 4900 1615
+Wire Wire Line
+	4900 1615 4615 1615
+Wire Wire Line
+	4615 1565 4615 1615
+Wire Wire Line
+	4615 1195 4900 1195
+Wire Wire Line
+	4615 1195 4615 1265
 Wire Wire Line
 	1455 1040 1455 1135
@@
 L Device:C C13
 U 1 1 615E1B36
-P 4520 1415
-F 0 "C13" H 4495 1320 50  0000 C CNN
-F 1 "100nF" V 4630 1415 50  0000 C CNN
-F 2 "Capacitor_SMD:C_1206_3216Metric_Pad1.33x1.80mm_HandSolder" H 4558 1265 50  0001 C CNN
-F 3 "~" H 4520 1415 50  0001 C CNN
-	1    4520 1415
+P 4900 1415
+F 0 "C13" H 4875 1320 50  0000 C CNN
+F 1 "100nF" V 5010 1415 50  0000 C CNN
+F 2 "Capacitor_SMD:C_1206_3216Metric_Pad1.33x1.80mm_HandSolder" H 4938 1265 50  0001 C CNN
+F 3 "~" H 4900 1415 50  0001 C CNN
+	1    4900 1415
 	-1   0    0    1
 $EndComp
@@
 L Device:C C11
 U 1 1 615E0997
-P 4235 1415
-F 0 "C11" H 4255 1330 50  0000 C CNN
-F 1 "1uF" V 4350 1415 50  0000 C CNN
-F 2 "Capacitor_SMD:C_1206_3216Metric_Pad1.33x1.80mm_HandSolder" H 4273 1265 50  0001 C CNN
-F 3 "~" H 4235 1415 50  0001 C CNN
-	1    4235 1415
-	-1   0    0    1
-$EndComp
-$Comp
-L Device:R R4
-U 1 1 615A8A09
-P 3475 1405
-F 0 "R4" V 3470 1450 50  0000 R CNN
-F 1 "2k/1w" V 3385 1530 50  0000 R CNN
-F 2 "Resistor_THT:R_Axial_DIN0414_L11.9mm_D4.5mm_P7.62mm_Vertical" V 3405 1405 50  0001 C CNN
-F 3 "~" H 3475 1405 50  0001 C CNN
-	1    3475 1405
+P 4615 1415
+F 0 "C11" H 4635 1330 50  0000 C CNN
+F 1 "1uF" V 4730 1415 50  0000 C CNN
+F 2 "Capacitor_SMD:C_1206_3216Metric_Pad1.33x1.80mm_HandSolder" H 4653 1265 50  0001 C CNN
+F 3 "~" H 4615 1415 50  0001 C CNN
+	1    4615 1415
 	-1   0    0    1
 $EndComp
@@
 L Device:CP C7
 U 1 1 6159A404
-P 3790 1425
-F 0 "C7" H 3908 1471 50  0000 L CNN
-F 1 "10uf/35v" H 3655 1330 50  0000 L CNN
-F 2 "Capacitor_THT:CP_Radial_D5.0mm_P2.50mm" H 3828 1275 50  0001 C CNN
-F 3 "~" H 3790 1425 50  0001 C CNN
-	1    3790 1425
+P 4170 1425
+F 0 "C7" H 4288 1471 50  0000 L CNN
+F 1 "10uf/35v" H 4035 1330 50  0000 L CNN
+F 2 "Capacitor_THT:CP_Radial_D5.0mm_P2.50mm" H 4208 1275 50  0001 C CNN
+F 3 "~" H 4170 1425 50  0001 C CNN
+	1    4170 1425
 	1    0    0    -1
 $EndComp
@@
 $EndComp
 $Comp
-L IGBT-DRIVER-rescue:miw06-24s24-GH-kicad U1
-U 1 1 6156C075
-P 2605 1025
-F 0 "U1" H 2855 1140 50  0000 C CNN
-F 1 "miw06-24s24" H 2855 1049 50  0000 C CNN
-F 2 "IGBT-DRIVER-emad:MIWI06" H 2605 1025 50  0001 C CNN
-F 3 "" H 2605 1025 50  0001 C CNN
-	1    2605 1025
-	1    0    0    -1
-$EndComp
-$Comp
 L Device:LED D9
 U 1 1 6196EC2F
@@
 	-1   0    0    1
 $EndComp
-Wire Wire Line
-	3475 1195 3790 1195
 Wire Notes Line width 12 style solid
 	6250 780  650  780
@@
 Wire Notes Line width 12 style solid
 	6250 780  6250 4565
-Wire Wire Line
-	3305 1615 3475 1615
 $Comp
 L power:GNDPWR #PWR012
@@
 Wire Wire Line
 	4575 3285 4515 3285
-$Sheet
-S 9080 2810 1010 1805
-U 6309618D
-F0 "Gate Driver Top" 50
-F1 "myGateDriver.sch" 50
-F2 "Pulse" I L 9080 3170 50
-F3 "Vpp" I R 10090 2860 50
-F4 "GND-d" I L 9080 3345 50
-F5 "Pulse-Disable" I R 10090 3000 50
-F6 "GND-p" I R 10090 4445 50
-F7 "Emitter" I R 10090 3965 50
-F8 "Gate" I R 10090 3795 50
-F9 "Collector" I R 10090 3605 50
-F10 "~Reset" I R 10090 3200 50
-F11 "~Fault" I R 10090 3395 50
-F12 "~its-ON" I R 10090 4195 50
-F13 "Pulse-Disable+" I L 9080 3715 50
-F14 "Pulse-Disable-" I L 9080 3855 50
-$EndSheet
 $Comp
 L Connector:Screw_Terminal_01x01 J3
@@
 Wire Wire Line
 	10090 3200 10550 3200
-Text Label 10550 2860 2    50   ~ 0
-VCC_top
-Wire Wire Line
-	10090 2860 10550 2860
 Text Label 10550 4445 2    50   ~ 0
 GND_top
@@
 Wire Wire Line
 	10135 6045 10775 6045
-Text Label 10690 5705 2    50   ~ 0
+Text Label 8550 5710 0    50   ~ 0
 VCC_BOTTOM
 Wire Wire Line
-	10135 5705 10690 5705
+	9125 5710 8550 5710
 Text Label 10775 7290 2    50   ~ 0
 GND_BOTTOM
@@
 F13 "Pulse-Disable+" I L 9125 6560 50
 F14 "Pulse-Disable-" I L 9125 6700 50
+F15 "Vin" I L 9125 5710 50
 $EndSheet
 Text Label 8585 3855 0    50   ~ 0
@@
 GND_top
 Wire Wire Line
-	3790 1195 4235 1195
-Connection ~ 3790 1195
-Connection ~ 4235 1195
-Wire Wire Line
-	4235 1615 3790 1615
-Connection ~ 4235 1615
-Connection ~ 3790 1615
+	4170 1195 4615 1195
+Connection ~ 4170 1195
+Connection ~ 4615 1195
+Wire Wire Line
+	4615 1615 4170 1615
+Connection ~ 4615 1615
+Connection ~ 4170 1615
 $Comp
 L power:+15V #PWR0101
@@
 	1    0    0    -1
 $EndComp
-$Comp
-L IGBT-DRIVER-rescue:miw06-24s24-GH-kicad U6
-U 1 1 61C3BFF7
-P 2670 5515
-F 0 "U6" H 2920 5630 50  0000 C CNN
-F 1 "miw06-24s24" H 2920 5539 50  0000 C CNN
-F 2 "IGBT-DRIVER-emad:MIWI06" H 2670 5515 50  0001 C CNN
-F 3 "" H 2670 5515 50  0001 C CNN
-	1    2670 5515
-	1    0    0    -1
-$EndComp
 Wire Wire Line
 	3540 5685 3855 5685
@@
 Text Label 4145 5685 2    50   ~ 0
 VCC_top
-Text Label 4235 1195 2    50   ~ 0
+Text Label 4615 1195 2    50   ~ 0
 VCC_BOTTOM
-Text Label 3975 1615 0    50   ~ 0
+Text Label 4355 1615 0    50   ~ 0
 GND_BOTTOM
 Text Label 3855 6105 0    50   ~ 0
@@
 	1    0    0    -1
 $EndComp
+$Comp
+L GateDriver:miw06-24s24 U7
+U 1 1 619584B7
+P 2605 1025
+F 0 "U7" H 2855 1140 50  0000 C CNN
+F 1 "miw06-24s24" H 2855 1049 50  0000 C CNN
+F 2 "IGBT-DRIVER-emad:MIWI06" H 2605 1025 50  0001 C CNN
+F 3 "" H 2605 1025 50  0001 C CNN
+	1    2605 1025
+	1    0    0    -1
+$EndComp
+$Comp
+L GateDriver:miw06-24s24 U8
+U 1 1 61959EFB
+P 2670 5515
+F 0 "U8" H 2920 5630 50  0000 C CNN
+F 1 "miw06-24s24" H 2920 5539 50  0000 C CNN
+F 2 "IGBT-DRIVER-emad:MIWI06" H 2670 5515 50  0001 C CNN
+F 3 "" H 2670 5515 50  0001 C CNN
+	1    2670 5515
+	1    0    0    -1
+$EndComp
+Wire Wire Line
+	9080 2925 8585 2925
+Text Label 8585 2925 0    50   ~ 0
+VCC_top
+NoConn ~ 10090 2860
+NoConn ~ 10135 5705
+Wire Wire Line
+	3475 1195 3650 1195
+Wire Wire Line
+	3305 1195 3475 1195
+Connection ~ 3475 1195
+Wire Wire Line
+	3475 1195 3475 1255
+Wire Wire Line
+	3305 1615 3475 1615
+Wire Wire Line
+	3475 1615 3650 1615
+Connection ~ 3475 1615
+Wire Wire Line
+	3475 1555 3475 1615
+$Comp
+L Device:R R4
+U 1 1 615A8A09
+P 3475 1405
+F 0 "R4" V 3470 1450 50  0000 R CNN
+F 1 "6k" V 3385 1530 50  0000 R CNN
+F 2 "Resistor_SMD:R_1206_3216Metric" V 3405 1405 50  0001 C CNN
+F 3 "~" H 3475 1405 50  0001 C CNN
+	1    3475 1405
+	-1   0    0    1
+$EndComp
+$Comp
+L Device:R R2
+U 1 1 61F6C95B
+P 3650 1405
+F 0 "R2" V 3645 1450 50  0000 R CNN
+F 1 "6k" V 3560 1530 50  0000 R CNN
+F 2 "Resistor_SMD:R_1206_3216Metric" V 3580 1405 50  0001 C CNN
+F 3 "~" H 3650 1405 50  0001 C CNN
+	1    3650 1405
+	-1   0    0    1
+$EndComp
+$Comp
+L Device:R R5
+U 1 1 61F70B28
+P 3820 1405
+F 0 "R5" V 3815 1450 50  0000 R CNN
+F 1 "6k" V 3730 1530 50  0000 R CNN
+F 2 "Resistor_SMD:R_1206_3216Metric" V 3750 1405 50  0001 C CNN
+F 3 "~" H 3820 1405 50  0001 C CNN
+	1    3820 1405
+	-1   0    0    1
+$EndComp
+Wire Wire Line
+	3650 1255 3650 1195
+Connection ~ 3650 1195
+Wire Wire Line
+	3650 1195 3820 1195
+Wire Wire Line
+	3820 1255 3820 1195
+Connection ~ 3820 1195
+Wire Wire Line
+	3820 1195 4170 1195
+Wire Wire Line
+	3650 1555 3650 1615
+Connection ~ 3650 1615
+Wire Wire Line
+	3650 1615 3820 1615
+Wire Wire Line
+	3820 1555 3820 1615
+Connection ~ 3820 1615
+Wire Wire Line
+	3820 1615 4170 1615
 $EndSCHEMATC

Commit message: placing back of bottom
Parts:
- removed H5: MountingHole, MountingHole:MountingHole_4.3x6.2mm_M4_Pad_Via, symbol Mechanical:MountingHole
- removed R10: 2k/1w, Resistor_THT:R_Axial_DIN0414_L11.9mm_D4.5mm_P7.62mm_Vertical, symbol Device:R
- added G1: LOGO, IGBT-DRIVER-emad:koalaLogo, symbol koalaLogo:LOGO
- added R7, R8, R9: 6k, Resistor_SMD:R_1206_3216Metric, symbol Device:R
Connections:
- net labels removed: pulse_disable_BOTTOM
- wire segments 123 -> 127
Other:
- moved on the sheet: C16, C17, C18, C19, C20, C8, H1, H2, H3, H4, J5, U8

Commit message: added top parts
Parts:
- removed C16, C4: 10uf/35v, Capacitor_THT:CP_Radial_D5.0mm_P2.50mm, symbol Device:CP
- removed D1, D9: LED, LED_SMD:LED_1206_3216Metric_Castellated, symbol Device:LED
- removed D29: DF10M, Diode_SMD:Diode_Bridge_Vishay_DFS, symbol Diode_Bridge:DF10M
- removed R3: 1.8k, Resistor_SMD:R_0805_2012Metric, symbol Device:R
- added BR1: DB107S, kicadFP:DIOB_DB107S, symbol MLC:DB107S
- added D2: LED_Green_0805, kicadFP:GREEN_LED_0805, symbol MLC:LED_Green_0805
- added LOGO1: Logo_Open_Hardware_Small, Symbol:OSHW-Logo_5.7x6mm_SilkScreen, symbol Graphic:Logo_Open_Hardware_Small
- IGBTSymbol1: symbol Graphic:SYM_Arrow45_Normal -> MLC:SKM200
- L1: renamed from L2; footprint Inductor_SMD:L_12x12mm_H6mm -> kicadFP:L_12x12mm_H6mm
- renumbered C8 to C1, C20 to C10, C13 to C12, C3 to C2, C17 to C4, C9 to C6, C18 to C7, C7 to C8, C19 to C9, H2 to H1, H3 to H2, H1 to H3, J3 to J2, J5 to J3, J6 to J4, J7 to J5, R7 to R1, R8 to R2, R4 to R3, R9 to R4, R2 to R5, R5 to R6, R1 to R7, U8 to U1, U7 to U2
Connections:
- net labels added: ON_Bottom
- net labels removed: +24V, GNDPWR, On_BOTTOM, pulse_disable_top
- wire segments 127 -> 116
Other:
- moved on the sheet: C1, C2, C6, C7, F1, J2, J3, J4, J5, L1

Commit message: topside added
Parts:
- added D24, D5: LED_Yellow_0805, kicadFP:LED_Yellow_0805, symbol MLC:LED_Yellow_0805
- added D44: LED_RED_0805, kicadFP:LED_RED_0805, symbol MLC:LED_RED_0805
- added R72, R73, R74: 1.8k, Resistor_SMD:R_0805_2012Metric, symbol Device:R
- D2: footprint kicadFP:GREEN_LED_0805 -> Diode_SMD:D_0805_2012Metric
Connections:
- net GNDD: now also D24.1 (K), D5.1 (K)
- net Pulse-BOTTOM: now also R73.2
- net Pulse-TOP: now also R72.2
- net Vin+: now also J1.9 (Pin_9), R74.2; no longer J1.6 (Pin_6)
- net at BR1.AC1, F1.2: now also D44.1 (K)
- net sheet61D91DB7/Collector renamed Gate Driver top/Collector
- new net: D5.2 (A), R72.1
- new net: D44.2 (A), R74.1
- new net: D24.2 (A), R73.1
- no-connect marks 2 -> 4
Changed lines of the file:
@@
 footrint check beshe
 Wire Wire Line
-	5750 3155 5680 3155
+	5750 3155 5715 3155
 Wire Wire Line
 	5280 3600 5280 3555
@@
 	-1   0    0    1
 $EndComp
-Text Label 6010 3155 0    50   ~ 0
+Text Label 6015 3155 0    50   ~ 0
 Vin+
 Text Label 4730 3155 2    50   ~ 0
 Vin-
-Text Label 3135 2900 2    50   ~ 0
+Text Label 1230 3100 0    50   ~ 0
 Vin+
 Text Label 3135 2800 2    50   ~ 0
@@
 	2365 2800 3135 2800
 Wire Wire Line
-	2365 2900 3135 2900
+	1865 3100 1230 3100
 Text Label 3130 2700 2    50   ~ 0
 Reset_top
@@
 Wire Wire Line
 	4730 3155 4880 3155
-Wire Wire Line
-	5950 3155 6010 3155
 $Comp
 L Connector:Screw_Terminal_01x01 J2
@@
 Wire Wire Line
 	12855 2905 12265 2905
-$Comp
-L MLC:LED_Green_0805 D2
-U 1 1 61D637F2
-P 5490 1670
-F 0 "D2" V 5536 1602 50  0000 R CNN
-F 1 "LED_Green_0805" V 5445 1602 50  0000 R CNN
-F 2 "kicadFP:GREEN_LED_0805" V 5490 1670 50  0001 C CNN
-F 3 "" V 5490 1670 50  0001 C CNN
-F 4 "MLCEL12237340" H 5490 1670 60  0001 C CNN "MLC"
-	1    5490 1670
-	0    -1   -1   0
-$EndComp
 Wire Wire Line
 	5490 1455 5490 1570
@@
 S 9125 1810 1010 1805
 U 61D91DC5
-F0 "sheet61D91DB7" 50
+F0 "Gate Driver top" 50
 F1 "myGateDriver.sch" 50
 F2 "Pulse" I L 9125 2170 50
@@
 Wire Wire Line
 	8555 2345 9125 2345
+Wire Wire Line
+	4610 4980 4610 4945
+$Comp
+L power:GNDD #PWR0103
+U 1 1 61A88EE7
+P 4610 5655
+F 0 "#PWR0103" H 4610 5405 50  0001 C CNN
+F 1 "GNDD" H 4614 5500 50  0000 C CNN
+F 2 "" H 4610 5655 50  0001 C CNN
+F 3 "" H 4610 5655 50  0001 C CNN
+	1    4610 5655
+	1    0    0    -1
+$EndComp
+Wire Wire Line
+	4610 5655 4610 5595
+$Comp
+L Device:R R72
+U 1 1 61A88EEE
+P 4610 5130
+F 0 "R72" V 4605 5125 50  0000 C CNN
+F 1 "1.8k" V 4494 5130 50  0000 C CNN
+F 2 "Resistor_SMD:R_0805_2012Metric" V 4540 5130 50  0001 C CNN
+F 3 "~" H 4610 5130 50  0001 C CNN
+	1    4610 5130
+	-1   0    0    1
+$EndComp
+Wire Wire Line
+	4610 5280 4610 5395
+$Comp
+L Device:R R74
+U 1 1 61AC73A2
+P 6000 2970
+F 0 "R74" V 5995 2965 50  0000 C CNN
+F 1 "1.8k" V 5884 2970 50  0000 C CNN
+F 2 "Resistor_SMD:R_0805_2012Metric" V 5930 2970 50  0001 C CNN
+F 3 "~" H 6000 2970 50  0001 C CNN
+	1    6000 2970
+	0    -1   -1   0
+$EndComp
+Wire Wire Line
+	5850 2970 5815 2970
+Wire Wire Line
+	6150 3155 6150 2970
+Wire Wire Line
+	5615 2970 5615 3065
+Wire Wire Line
+	5615 3065 5715 3065
+Wire Wire Line
+	5715 3065 5715 3155
+Connection ~ 5715 3155
+Wire Wire Line
+	5715 3155 5680 3155
+$Comp
+L MLC:LED_Yellow_0805 D5
+U 1 1 61B1EC6B
+P 4610 5495
+F 0 "D5" V 4656 5427 50  0000 R CNN
+F 1 "LED_Yellow_0805" H 5035 5625 50  0000 R CNN
+F 2 "kicadFP:LED_Yellow_0805" V 4610 5495 50  0001 C CNN
+F 3 "" V 4610 5495 50  0001 C CNN
+F 4 "MLCEL12237704" H 4610 5495 60  0001 C CNN "MLC"
+	1    4610 5495
+	0    -1   -1   0
+$EndComp
+Text Label 4610 4945 2    50   ~ 0
+Pulse-TOP
+Wire Wire Line
+	4985 4985 4985 4950
+$Comp
+L power:GNDD #PWR0104
+U 1 1 61B271F8
+P 4985 5660
+F 0 "#PWR0104" H 4985 5410 50  0001 C CNN
+F 1 "GNDD" H 4989 5505 50  0000 C CNN
+F 2 "" H 4985 5660 50  0001 C CNN
+F 3 "" H 4985 5660 50  0001 C CNN
+	1    4985 5660
+	1    0    0    -1
+$EndComp
+Wire Wire Line
+	4985 5660 4985 5600
+$Comp
+L Device:R R73
+U 1 1 61B271FF
+P 4985 5135
+F 0 "R73" V 4980 5130 50  0000 C CNN
+F 1 "1.8k" V 4869 5135 50  0000 C CNN
+F 2 "Resistor_SMD:R_0805_2012Metric" V 4915 5135 50  0001 C CNN
+F 3 "~" H 4985 5135 50  0001 C CNN
+	1    4985 5135
+	-1   0    0    1
+$EndComp
+Wire Wire Line
+	4985 5285 4985 5400
+$Comp
+L MLC:LED_Yellow_0805 D24
+U 1 1 61B27207
+P 4985 5500
+F 0 "D24" V 5031 5432 50  0000 R CNN
+F 1 "LED_Yellow_0805" H 5405 5635 50  0000 R CNN
+F 2 "kicadFP:LED_Yellow_0805" V 4985 5500 50  0001 C CNN
+F 3 "" V 4985 5500 50  0001 C CNN
+F 4 "MLCEL12237704" H 4985 5500 60  0001 C CNN "MLC"
+	1    4985 5500
+	0    -1   -1   0
+$EndComp
+Text Label 4985 4950 0    50   ~ 0
+Pulse-BOTTOM
+$Comp
+L MLC:LED_RED_0805 D44
+U 1 1 61B45156
+P 5715 2970
+F 0 "D44" H 5715 3205 50  0000 C CNN
+F 1 "LED_RED_0805" H 5715 3114 50  0000 C CNN
+F 2 "kicadFP:LED_RED_0805" V 5715 2970 50  0001 C CNN
+F 3 "" V 5715 2970 50  0001 C CNN
+F 4 "MLCEL12237862" H 5715 2970 60  0001 C CNN "MLC"
+	1    5715 2970
+	1    0    0    -1
+$EndComp
+Wire Wire Line
+	5950 3155 6150 3155
+NoConn ~ 2365 3100
+NoConn ~ 2365 2900
+$Comp
+L MLC:LED_Green_0805 D2
+U 1 1 61B99539
+P 5490 1670
+F 0 "D2" V 5536 1602 50  0000 R CNN
+F 1 "LED_Green_0805" V 5445 1602 50  0000 R CNN
+F 2 "Diode_SMD:D_0805_2012Metric" V 5490 1670 50  0001 C CNN
+F 3 "" V 5490 1670 50  0001 C CNN
+F 4 "MLCEL12237340" H 5490 1670 60  0001 C CNN "MLC"
+	1    5490 1670
+	0    -1   -1   0
+$EndComp
 $EndSCHEMATC
