File: IGBT DRIVER.sch (KiCad schematic (older format))
At the start: 41 parts, among them J1 Conn_02x05_Odd_Even, J2 Screw_Terminal_01x01, J3 Screw_Terminal_01x01, J4 Conn_01x02, J5 Conn_01x02, U1 miw06-24s24, U2 miw06-24s24

Commit message: yii
Parts:
- D2: footprint Diode_SMD:D_0805_2012Metric -> kicadFP:LED_Green_0805
Changed lines of the file:
@@
 $Comp
 L MLC:LED_Green_0805 D2
-U 1 1 61B99539
+U 1 1 61B8A52C
 P 5490 1670
 F 0 "D2" V 5536 1602 50  0000 R CNN
 F 1 "LED_Green_0805" V 5445 1602 50  0000 R CNN
-F 2 "Diode_SMD:D_0805_2012Metric" V 5490 1670 50  0001 C CNN
+F 2 "kicadFP:LED_Green_0805" V 5490 1670 50  0001 C CNN
 F 3 "" V 5490 1670 50  0001 C CNN
 F 4 "MLCEL12237340" H 5490 1670 60  0001 C CNN "MLC"

Commit message: 15v logic added
Parts:
- added U11: L7833s(D2pack), Package_TO_SOT_SMD:TO-263-3_TabPin2, symbol MLC:L7805(D2pack)
- J1: footprint Connector_IDC:IDC-Header_2x05-1MP_P2.54mm_Latch_Horizontal -> kicadFP:IDC-Header_2x05-1MP_P2.54mm_Latch_Horizontal
Connections:
- net +15V: now also U11.1 (IN)
- net GNDD: now also U11.2 (GND)
- new net +5V: U11.3 (OUT)
Changed lines of the file:
@@
 F12 "~Pulse-Disable" I L 12855 2730 50
 F13 "its-ON" I L 12855 2905 50
+F14 "Vccmin" I L 12855 3165 50
 $EndSheet
 Wire Wire Line
@@
 F 0 "J1" H 2115 3317 50  0000 C CNN
 F 1 "Conn_02x05_Odd_Even" H 2115 3226 50  0000 C CNN
-F 2 "Connector_IDC:IDC-Header_2x05-1MP_P2.54mm_Latch_Horizontal" H 2065 2900 50  0001 C CNN
+F 2 "kicadFP:IDC-Header_2x05-1MP_P2.54mm_Latch_Horizontal" H 2065 2900 50  0001 C CNN
 F 3 "~" H 2065 2900 50  0001 C CNN
 	1    2065 2900
@@
 F12 "~Pulse-Disable" I L 9125 2735 50
 F13 "its-ON" I L 9125 2910 50
+F14 "Vccmin" I L 9125 3125 50
 $EndSheet
 Text Label 8615 2735 0    50   ~ 0
@@
 	0    -1   -1   0
 $EndComp
+$Comp
+L MLC:L7805(D2pack) U11
+U 1 1 61A06489
+P 3095 6735
+F 0 "U11" H 3095 6977 50  0000 C CNN
+F 1 "L7833s(D2pack)" H 3095 6886 50  0000 C CNN
+F 2 "Package_TO_SOT_SMD:TO-263-3_TabPin2" H 3120 6585 50  0001 L CIN
+F 3 "" H 3095 6685 50  0001 C CNN
+F 4 "MLCEL12238271" H 3095 6735 60  0001 C CNN "MLC"
+	1    3095 6735
+	1    0    0    -1
+$EndComp
+$Comp
+L power:+15V #PWR0105
+U 1 1 61A07A43
+P 2525 6735
+F 0 "#PWR0105" H 2525 6585 50  0001 C CNN
+F 1 "+15V" H 2540 6908 50  0000 C CNN
+F 2 "" H 2525 6735 50  0001 C CNN
+F 3 "" H 2525 6735 50  0001 C CNN
+	1    2525 6735
+	1    0    0    -1
+$EndComp
+Wire Wire Line
+	2795 6735 2525 6735
+$Comp
+L power:GNDD #PWR0106
+U 1 1 61A15C37
+P 3095 7095
+F 0 "#PWR0106" H 3095 6845 50  0001 C CNN
+F 1 "GNDD" H 3099 6940 50  0000 C CNN
+F 2 "" H 3095 7095 50  0001 C CNN
+F 3 "" H 3095 7095 50  0001 C CNN
+	1    3095 7095
+	1    0    0    -1
+$EndComp
+Wire Wire Line
+	3095 7095 3095 7035
+$Comp
+L power:+5V #PWR0107
+U 1 1 61A1C064
+P 3560 6735
+F 0 "#PWR0107" H 3560 6585 50  0001 C CNN
+F 1 "+5V" H 3575 6908 50  0000 C CNN
+F 2 "" H 3560 6735 50  0001 C CNN
+F 3 "" H 3560 6735 50  0001 C CNN
+	1    3560 6735
+	1    0    0    -1
+$EndComp
+Wire Wire Line
+	3395 6735 3560 6735
+$Comp
+L power:+5V #PWR0108
+U 1 1 61A63744
+P 9000 3120
+F 0 "#PWR0108" H 9000 2970 50  0001 C CNN
+F 1 "+5V" H 9015 3293 50  0000 C CNN
+F 2 "" H 9000 3120 50  0001 C CNN
+F 3 "" H 9000 3120 50  0001 C CNN
+	1    9000 3120
+	1    0    0    -1
+$EndComp
+Wire Wire Line
+	9125 3125 9000 3125
+Wire Wire Line
+	9000 3125 9000 3120
+$Comp
+L power:+5V #PWR0109
+U 1 1 61A69C82
+P 12680 3165
+F 0 "#PWR0109" H 12680 3015 50  0001 C CNN
+F 1 "+5V" H 12695 3338 50  0000 C CNN
+F 2 "" H 12680 3165 50  0001 C CNN
+F 3 "" H 12680 3165 50  0001 C CNN
+	1    12680 3165
+	1    0    0    -1
+$EndComp
+Wire Wire Line
+	12855 3165 12680 3165
 $EndSCHEMATC
