File: myGateDriver.sch (KiCad schematic (older format))
At the start: 92 parts, among them Q1 BC817, Q2 BC817, Q3 BC817, Q4 BC807, Q5 BC817, Q6 BC817, Q7 BC817, Q8 d44vh10, Q9 D45VH10, U1 PC817, U2 6N136S, U3 PC817

Commit message: some placements have done
Parts:
- removed C21: 47uf/35v, Capacitor_THT:CP_Radial_D8.0mm_P3.80mm, symbol Device:CP
- removed C22: 100nF, Capacitor_SMD:C_0805_2012Metric, symbol Device:C
- removed D4: 1.5KE14A, Diode_THT:D_DO-201AD_P15.24mm_Horizontal, symbol Diode:1.5KExxA
- removed D6: 1.5KE6V8A, Diode_THT:D_DO-201AD_P15.24mm_Horizontal, symbol Diode:1.5KExxA
- removed DStatic1, DStatic2, DStatic3, DStatic4, DStatic5, DzDynamic1: 1.5KE160A, Diode_THT:D_DO-201AD_P15.24mm_Horizontal, symbol Diode:1.5KExxA
- added D16, D17, D18, D19, D20, D21: SMCJ160CA-13-F, IGBT-DRIVER-emad:DIOM7959X250N, symbol SMCJ160CA-13-F:SMCJ160CA-13-F
- added R6: 1.5k, Resistor_SMD:R_0805_2012Metric, symbol Device:R
- added Rex?: 1k, Resistor_SMD:R_0805_2012Metric, symbol Device:R
- added U?: ps2801, SOP-4_4.4x2.6mm_P1.27mm, symbol Isolator:PC817
- CDynamic1: value 100nF -> 100nF 250v; footprint Capacitor_THT:C_Rect_L16.5mm_W6.0mm_P15.00mm_MKT -> Capacitor_THT:C_Rect_L13.0mm_W4.0mm_P10.00mm_FKS3_FKP3_MKS4
- D3, DzSaturation1: footprint Diode_THT:D_DO-201AD_P5.08mm_Vertical_AnodeUp -> Diode_SMD:D_MELF
- D5: footprint Diode_THT:D_DO-201AD_P15.24mm_Horizontal -> Diode_THT:D_DO-35_SOD27_P7.62mm_Horizontal
- D7: value 26v TVS -> 26v Zener
- F2: footprint Fuse:Fuse_Schurter_UMZ250 -> IGBT-DRIVER-emad:fuse.holder.1808
- R6: value 3.3k-1/4W -> 1.8k; footprint Resistor_THT:R_Axial_DIN0207_L6.3mm_D2.5mm_P10.16mm_Horizontal -> Resistor_SMD:R_0805_2012Metric
- Rex5: footprint Resistor_THT:R_Axial_DIN0207_L6.3mm_D2.5mm_P10.16mm_Horizontal -> Resistor_SMD:R_0805_2012Metric
- U1, U3: value PC817 -> ps2801; footprint Package_DIP:DIP-4_W7.62mm -> SOP-4_4.4x2.6mm_P1.27mm
Connections:
- net labels added: fault
- wire segments 279 -> 269
Other:
- moved on the sheet: D15, R16

Commit message: placing back of bottom
Parts:
- removed F3: Fuse_Small, IGBT-DRIVER-emad:fuse.holder.1808, symbol Device:Fuse_Small
- removed U3: ps2801, SOP-4_4.4x2.6mm_P1.27mm, symbol Isolator:PC817
- added C2: 100nF, Capacitor_SMD:C_1206_3216Metric_Pad1.33x1.80mm_HandSolder, symbol Device:C
- added D3: SMCJ7A, IGBT-DRIVER-emad:DIOM7959X250N, symbol SMCJ160CA-13-F:SMCJ160CA-13-F
- added Rex2: 1k, Resistor_SMD:R_0805_2012Metric, symbol Device:R
- added U2: ps2801, SOP-4_4.4x2.6mm_P1.27mm, symbol Isolator:PC817
- C1: footprint Capacitor_SMD:C_0805_2012Metric -> Capacitor_SMD:C_1206_3216Metric_Pad1.33x1.80mm_HandSolder
- D2: value 1.5KE4A -> Dz4v; footprint Diode_THT:D_DO-201AD_P5.08mm_Vertical_AnodeUp -> Diode_SMD:D_MELF
- gave numbers to parts that had none: 2
Connections:
- net labels added: ItsOn, its-ON, ~Pulse-Disable
- net labels removed: GNDPWR, Pulse-Disable+, Pulse-Disable-, ~its-ON
- wire segments 269 -> 276
- no-connect marks 0 -> 1
Other:
- note added: "find an optocoupler without base pin to tollerate high noise enviorments"
- moved on the sheet: R23, Rex1, U1, U6

Commit message: a
Other:
- moved on the sheet: C15, D15, D22, Dex7, F4, Q18, R16, R18, R19, R6

Commit message: added top parts
Parts:
- added D1: LED_RED_0805, kicadFP:LED_RED_0805_2012Metric, symbol MLC:LED_RED_0805
- added D12: 1n4148, Diode_SMD:D_SMA, symbol Device:D_Schottky
- added D23: LED_Blue_0805, kicadFP:LED_BLUE_0805, symbol MLC:LED_Blue_0805
- added R37: 20K, Resistor_SMD:R_0805_2012Metric, symbol Device:R
- added R39: 220, Resistor_SMD:R_0805_2012Metric, symbol Device:R
- added R40: 1k, Resistor_SMD:R_0805_2012Metric, symbol Device:R
- R38: renamed from RClamp1; value 10K -> 20K
- U4, U5: renamed from U1; footprint SOP-4_4.4x2.6mm_P1.27mm -> Package_SO:SOP-4_4.4x2.6mm_P1.27mm
- U6: renamed from U2; footprint SOP-4_4.4x2.6mm_P1.27mm -> Package_SO:SOP-4_4.4x2.6mm_P1.27mm
- renumbered C2 to C13, C10 to C14, C25 to C15, C26 to C16, C27 to C17, C28 to C18, C29 to C19, C30 to C20, C31 to C21, C32 to C22, C33 to C23, C34 to C24, C35 to C25, C36 to C26, C37 to C27, C38 to C28, Cex1 to C29, CDynamic1 to C30, C39 to C31, C40 to C32, C1 to C33, C2 to C34, CShortPulseFilter1 to C35, CblankTime1 to C36, Cex2 to C37, CsoftTurnOffTiming1 to C38, C5 to C39, CsoftTurnOff2 to C40, Cclamp1 to C41, D3 to D10, D21 to D11, D3 to D13, D7 to D14, D5 to D15, DzSaturation1 to D16, Dex1 to D17, Dex2 to D18, DZunderVoltageFault1 to D19, Dex5 to D20, DprotectionHigh1 to D21, DprotectionLow1 to D22, D16 to D4, D2 to D5, D17 to D6, D18 to D7, D19 to D8, D20 to D9, Q6 to Q10, Q8 to Q11, Q9 to Q12, QfaultLatch1 to Q2, QsoftTurnOnn1 to Q3, Q2 to Q4, Q7 to Q5, Qclamp1 to Q6, Q3 to Q7, Q5 to Q8, Q4 to Q9, R20 to R10, Rex1 to R11, RDynamic1 to R12, Rex1 to R13, Rex2 to R14, R7 to R15, RshortPulseFilter1 to R16, Rex3 to R17, RBlankTime1 to R18, Rex4 to R19, R5 to R20, Rex5 to R21, Rex2 to R22, RSofTurnoffTiming1 to R23, Rex6 to R24, RAfterfaultTurnOnDelay1 to R25, R6 to R26, R6 to R27, R8 to R28, R9 to R29, Rex7 to R30, R11 to R31, RsoftTurnoff2 to R32, Ron1 to R33, Roff1 to R34, Ron4 to R35, Roff3 to R36, R2 to R9, U2 to U3
Connections:
- net Emitter: now also R37.1
- net GND-p: now also D23.1 (K); no longer U4.2
- net Gate: now also R37.2
- net Vpp: now also R13.2, R39.1, R40.2
- net fault: now also U4.2, D1.1 (K), D12.1 (K); no longer R13.2
- net at U3.7: now also D12.2 (A)
- new net: D23.2 (A), R39.2
- new net: D1.2 (A), R40.1
- no-connect marks 1 -> 0
Other:
- moved on the sheet: R45, R59, R60, R62, U10

Commit message: topside added
Parts:
- removed D5: Dz4v, Diode_SMD:D_MELF, symbol Diode:1.5KExxA
- D1: footprint kicadFP:LED_RED_0805_2012Metric -> kicadFP:LED_RED_0805
Connections:
- net Pulse: now also R9.2
- net at D12.2 (A): now also R16.2, U3.6; no longer U3.7
Other:
- moved on the sheet: D7, R40

Commit message: 15v logic added
Parts:
- added JP2: SolderJumper_3_Bridged12, Jumper:SolderJumper-3_P1.3mm_Bridged2Bar12_Pad1.0x1.5mm, symbol Jumper:SolderJumper_3_Bridged12
Connections:
- net GND-d: now also JP2.3 (B); no longer U3.3
- new net: JP2.2 (C), U3.3
- new net Vccmin: JP2.1 (A)
Other:
- note added: "jumper for 15v logic"
Changed lines of the file:
@@
 	0    1    1    0
 $EndComp
-Wire Wire Line
-	1995 9130 2115 9130
 $Comp
 L Device:R R?
@@
 Text HLabel 6190 6470 1    50   Input ~ 0
 Vpp
-Text HLabel 1995 9130 0    50   Input ~ 0
+Text HLabel 1635 9580 0    50   Input ~ 0
 GND-d
 Text HLabel 2075 8870 1    50   Input ~ 0
@@
 Wire Wire Line
 	1945 1510 1945 1500
+$Comp
+L Jumper:SolderJumper_3_Bridged12 JP2
+U 1 1 61A28ABF
+P 1870 9580
+AR Path="/61D91DC5/61A28ABF" Ref="JP2"  Part="1"
+AR Path="/6340E1F3/61A28ABF" Ref="JP1"  Part="1"
+F 0 "JP2" H 1870 9693 50  0000 C CNN
+F 1 "SolderJumper_3_Bridged12" H 1870 9784 50  0000 C CNN
+F 2 "Jumper:SolderJumper-3_P1.3mm_Bridged2Bar12_Pad1.0x1.5mm" H 1870 9580 50  0001 C CNN
+F 3 "~" H 1870 9580 50  0001 C CNN
+	1    1870 9580
+	-1   0    0    1
+$EndComp
+Wire Wire Line
+	1635 9580 1670 9580
+Text HLabel 2070 9580 2    50   Input ~ 0
+Vccmin
+Wire Wire Line
+	1870 9430 1870 9130
+Wire Wire Line
+	1870 9130 2115 9130
+Text Notes 965  9535 0    50   ~ 0
+jumper for 15v logic
 $EndSCHEMATC

Commit message: soft shutdown wiki pic added
Connections:
- net on: no longer Q8.1 (B), Q9.1 (B)
Other:
- moved on the sheet: C39, C40, C41, D18, D19, D21, D22, Q11, Q12, Q5, Q8, Q9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
