File: myGateDriver.sch (KiCad schematic (older format))
At the start: 99 parts, among them Q1 BC817, Q10 BC817, Q11 d44vh10, Q12 D45VH10, Q2 BC807, Q3 BC817, Q4 BC817, Q5 BC817, Q6 BUK7880-55A, Q7 BC817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

Commit message: .
Parts:
- D16: value Dz10v -> Dz13v
Connections:
- net on: now also Q8.1 (B), Q9.1 (B)
Other:
- moved on the sheet: D1, D15, R19, R40
